File: PCBA-FLUX-01A/BlockDiagram.kicad_sch (KiCad schematic)
At the start: 0 parts

Commit message: Finished inverter design and started working on MCU pin out
Other:
- company: (none) -> Jovanovski Laboratory - JLAB
