File: PCBA-FLUX-01A/RevisionHistory.kicad_sch (KiCad schematic)
At the start: 0 parts

Commit message: Finished inverter design and started working on MCU pin out
Other:
- company: (none) -> Jovanovski Laboratory - JLAB
Changed lines of the file:
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@@
 	(generator_version "10.0")
 	(paper "A4")
+	(title_block
+		(rev "1.0.0")
+		(company "Jovanovski Laboratory - JLAB")
+		(comment 1 "Bvrny")
+		(comment 2 "Nikola Jovanovski")
+		(comment 3 "Flux")
+		(comment 4 "Vortex")
+	)
 )
