File: PCBA-FLUX-01A/PCBA-FLUX-01A.kicad_sch (KiCad schematic)
At the start: 0 parts

Commit message: Changes were made
Other:
- note added: "2026-07-06"
- note removed: "2026-05-26"
Changed lines of the file:
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@@
 		)
 	)
-	(text "2026-05-26"
+	(text "2026-07-06"
 		(exclude_from_sim no)
 		(at 388.62 35.687 0)

Commit message: Finished schematic?
Other:
- note removed: "Power Input"
Changed lines of the file:
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@@
 		(company "Jovanovski Laboratory - JLAB")
 		(comment 1 "Bvrny")
-		(comment 2 "Nikola Jovanovski")
 		(comment 3 "Flux")
 		(comment 4 "Vortex")
 	)
-	(text "Phase V\n"
+	(text "Phase W"
 		(exclude_from_sim no)
 		(at 45.72 116.967 0)
@@
 		)
 	)
-	(text "Power Input"
+	(text "Phase U\n"
 		(exclude_from_sim no)
 		(at 45.72 101.727 0)
@@
 		)
 	)
-	(text "Phase U"
+	(text "Phase V"
 		(exclude_from_sim no)
 		(at 45.72 109.347 0)
@@
 		)
 	)
-	(text "Phase W\n"
+	(text "..............."
 		(exclude_from_sim no)
 		(at 45.72 124.587 0)
