File: PCBA-FLUX-01A/PCBA-FLUX-01A.kicad_pcb (KiCad board)
At the start: 2 copper layers, 0 parts

Commit message: Started with Flux layout
Parts:
- added C104: C, Capacitor_THT:C_Rect_L9.0mm_W6.4mm_P7.50mm_MKT, F.Cu at (105.1, 115.0)
- added C105: C, Capacitor_THT:C_Rect_L9.0mm_W6.4mm_P7.50mm_MKT, F.Cu at (159.9, 115.0)
- added C106: C, Capacitor_THT:C_Rect_L9.0mm_W6.4mm_P7.50mm_MKT, F.Cu at (214.7, 114.9)
- added C107: 1000uF, Capacitor_THT:CP_Radial_D18.0mm_P7.50mm, F.Cu at (159.0, 27.0)
- added C108: 1000uF, Capacitor_THT:CP_Radial_D18.0mm_P7.50mm, F.Cu at (192.1, 64.8)
- added C109: 1000uF, Capacitor_THT:CP_Radial_D18.0mm_P7.50mm, F.Cu at (210.6, 64.8)
- added C110: 1000uF, Capacitor_THT:CP_Radial_D18.0mm_P7.50mm, F.Cu at (28.3, 68.1)
- added C111: 1000uF, Capacitor_THT:CP_Radial_D18.0mm_P7.50mm, F.Cu at (235.6, 78.4)
- added C112: 10uF, Capacitor_SMD:C_1210_3225Metric, F.Cu at (72.3, 134.9)
- added C113: 10uF, Capacitor_SMD:C_1210_3225Metric, F.Cu at (72.3, 131.6)
- added C114: 10uF, Capacitor_SMD:C_1210_3225Metric, F.Cu at (72.3, 128.4)
- added C115: 10uF, Capacitor_SMD:C_1210_3225Metric, F.Cu at (72.3, 148.8)
- added C116: 10uF, Capacitor_SMD:C_1210_3225Metric, F.Cu at (72.3, 114.4)
- added C117: 100nF, Capacitor_SMD:C_0805_2012Metric, F.Cu at (68.9, 153.7)
- added C118: 1000uF, Capacitor_THT:CP_Radial_D18.0mm_P7.50mm, F.Cu at (149.3, 64.6)
- added C119: 10uF, Capacitor_SMD:C_1210_3225Metric, F.Cu at (127.1, 148.8)
- added C120: 1000uF, Capacitor_THT:CP_Radial_D18.0mm_P7.50mm, F.Cu at (69.2, 64.8)
- added C121: 10uF, Capacitor_SMD:C_1210_3225Metric, F.Cu at (127.1, 134.8)
- added C122: 1000uF, Capacitor_THT:CP_Radial_D18.0mm_P7.50mm, F.Cu at (87.7, 64.8)
- added C123: 10uF, Capacitor_SMD:C_1210_3225Metric, F.Cu at (127.1, 131.6)
- added C124: 1000uF, Capacitor_THT:CP_Radial_D18.0mm_P7.50mm, F.Cu at (130.8, 64.6)
- added C125: 10uF, Capacitor_SMD:C_1210_3225Metric, F.Cu at (127.1, 114.3)
- added C126: 1000uF, Capacitor_THT:CP_Radial_D18.0mm_P7.50mm, F.Cu at (215.1, 28.8)
- added C127: 10uF, Capacitor_SMD:C_1210_3225Metric, F.Cu at (127.1, 128.3)
- added C128: 100nF, Capacitor_SMD:C_0805_2012Metric, F.Cu at (121.7, 153.6)
- added C129: 1000uF, Capacitor_THT:CP_Radial_D18.0mm_P7.50mm, F.Cu at (116.2, 17.2)
- added C130: 10uF, Capacitor_SMD:C_1210_3225Metric, F.Cu at (181.9, 148.7)
- added C131: 1000uF, Capacitor_THT:CP_Radial_D18.0mm_P7.50mm, F.Cu at (135.8, 17.2)
- added C132: 10uF, Capacitor_SMD:C_1210_3225Metric, F.Cu at (181.9, 114.3)
- added C133: 1000uF, Capacitor_THT:CP_Radial_D18.0mm_P7.50mm, F.Cu at (155.3, 17.2)
- added C134: 10uF, Capacitor_SMD:C_1210_3225Metric, F.Cu at (181.9, 134.8)
- added C135: 1000uF, Capacitor_THT:CP_Radial_D18.0mm_P7.50mm, F.Cu at (174.9, 17.2)
- added C136: 10uF, Capacitor_SMD:C_1210_3225Metric, F.Cu at (181.9, 131.6)
- added C137: 1000uF, Capacitor_THT:CP_Radial_D18.0mm_P7.50mm, F.Cu at (197.7, 12.7)
- added C138: 10uF, Capacitor_SMD:C_1210_3225Metric, F.Cu at (181.8, 128.3)
- added C139: 100nF, Capacitor_SMD:C_0805_2012Metric, F.Cu at (178.5, 153.6)
- added C140: 10uF, Capacitor_SMD:C_1210_3225Metric, F.Cu at (127.1, 111.1)
- added C141: 10uF, Capacitor_SMD:C_1210_3225Metric, F.Cu at (127.1, 152.0)
- added C142: 100nF, Capacitor_SMD:C_0805_2012Metric, F.Cu at (119.7, 153.6)
- added C29: 100nF, Capacitor_SMD:C_0402_1005Metric, F.Cu at (91.0, 100.5)
- added C30: 100nF, Capacitor_SMD:C_0402_1005Metric, F.Cu at (99.5, 100.5)
- added C31: 22uF, Capacitor_SMD:C_1206_3216Metric, F.Cu at (91.3, 152.9)
- added C32: 22uF, Capacitor_SMD:C_1206_3216Metric, F.Cu at (91.3, 150.5)
- added C33: 1nF, Capacitor_SMD:C_0603_1608Metric, F.Cu at (97.6, 160.4)
- added C34: 1nF, Capacitor_SMD:C_0603_1608Metric, F.Cu at (97.6, 155.8)
- added C35: 100nF, Capacitor_SMD:C_0402_1005Metric, F.Cu at (87.6, 154.3)
- added C36: 2.2nF, Capacitor_SMD:C_0603_1608Metric, F.Cu at (100.5, 104.0)
- added C37: 2.2uF, Capacitor_SMD:C_1206_3216Metric, F.Cu at (87.4, 157.2)
- added C38: 100nF, Capacitor_SMD:C_0402_1005Metric, F.Cu at (85.2, 158.7)
- added C39: 3.3nF, Capacitor_SMD:C_0603_1608Metric, F.Cu at (97.0, 94.2)
- added C40: 100nF, Capacitor_SMD:C_0402_1005Metric, F.Cu at (92.5, 88.0)
- added C41: 1nF, Capacitor_SMD:C_0603_1608Metric, F.Cu at (96.2, 90.8)
- added C42: 22uF, Capacitor_SMD:C_1206_3216Metric, F.Cu at (146.1, 152.8)
- added C43: 100nF, Capacitor_SMD:C_0805_2012Metric, F.Cu at (64.9, 153.7)
- added C44: 100nF, Capacitor_SMD:C_0402_1005Metric, F.Cu at (154.3, 100.5)
- added C45: 100nF, Capacitor_SMD:C_0805_2012Metric, F.Cu at (66.9, 109.5)
- added C46: 22uF, Capacitor_SMD:C_1206_3216Metric, F.Cu at (146.1, 150.4)
- added C47: 100nF, Capacitor_SMD:C_0805_2012Metric, F.Cu at (66.9, 153.7)
- added C48: 100nF, Capacitor_SMD:C_0402_1005Metric, F.Cu at (90.6, 182.2)
- added C49: 100nF, Capacitor_SMD:C_0402_1005Metric, F.Cu at (145.8, 100.5)
- added C50: 100nF, Capacitor_SMD:C_0805_2012Metric, F.Cu at (68.9, 109.5)
- added C51: 1nF, Capacitor_SMD:C_0603_1608Metric, F.Cu at (152.6, 160.4)
- added C52: 1nF, Capacitor_SMD:C_0603_1608Metric, F.Cu at (152.6, 155.8)
- added C53: 100nF, Capacitor_SMD:C_0402_1005Metric, F.Cu at (142.4, 154.2)
- added C54: 2.2uF, Capacitor_SMD:C_1206_3216Metric, F.Cu at (142.2, 157.1)
- added C55: 2.2nF, Capacitor_SMD:C_0603_1608Metric, F.Cu at (155.3, 103.9)
- added C56: 100nF, Capacitor_SMD:C_0402_1005Metric, F.Cu at (140.1, 158.6)
- added C57: 3.3nF, Capacitor_SMD:C_0603_1608Metric, F.Cu at (151.8, 94.1)
- added C58: 100nF, Capacitor_SMD:C_0402_1005Metric, F.Cu at (147.3, 88.0)
- added C59: 1nF, Capacitor_SMD:C_0603_1608Metric, F.Cu at (151.0, 90.7)
- added C60: 100nF, Capacitor_SMD:C_0805_2012Metric, F.Cu at (121.7, 109.4)
- added C61: 100nF, Capacitor_SMD:C_0805_2012Metric, F.Cu at (119.7, 109.4)
- added C62: 100nF, Capacitor_SMD:C_0805_2012Metric, F.Cu at (123.7, 109.4)
- added C63: 100nF, Capacitor_SMD:C_0402_1005Metric, F.Cu at (48.1, 169.6)
- added C64: 100nF, Capacitor_SMD:C_0805_2012Metric, F.Cu at (123.8, 153.6)
- added C65: 22uF, Capacitor_SMD:C_1206_3216Metric, F.Cu at (200.9, 152.8)
- added C66: 100nF, Capacitor_SMD:C_0402_1005Metric, F.Cu at (200.7, 100.5)
- added C67: 22uF, Capacitor_SMD:C_1206_3216Metric, F.Cu at (200.9, 150.4)
- added C68: 100nF, Capacitor_SMD:C_0402_1005Metric, F.Cu at (209.2, 100.5)
- added C69: 1nF, Capacitor_SMD:C_0603_1608Metric, F.Cu at (207.2, 160.3)
- added C70: 1nF, Capacitor_SMD:C_0603_1608Metric, F.Cu at (207.2, 155.8)
- added C71: 100nF, Capacitor_SMD:C_0402_1005Metric, F.Cu at (197.2, 154.2)
- added C72: 2.2uF, Capacitor_SMD:C_1206_3216Metric, F.Cu at (197.0, 157.1)
- added C73: 2.2nF, Capacitor_SMD:C_0603_1608Metric, F.Cu at (210.2, 103.9)
- added C74: 100nF, Capacitor_SMD:C_0402_1005Metric, F.Cu at (194.8, 158.6)
- added C75: 3.3nF, Capacitor_SMD:C_0603_1608Metric, F.Cu at (206.7, 94.2)
- added C76: 100nF, Capacitor_SMD:C_0402_1005Metric, F.Cu at (202.2, 88.0)
- added C77: 1nF, Capacitor_SMD:C_0603_1608Metric, F.Cu at (206.7, 94.2)
- added C78: 100nF, Capacitor_SMD:C_0805_2012Metric, F.Cu at (174.5, 153.6)
- added C79: 100nF, Capacitor_SMD:C_0805_2012Metric, F.Cu at (176.5, 153.6)
- added C80: 100nF, Capacitor_SMD:C_0805_2012Metric, F.Cu at (176.5, 109.4)
- added C81: 100nF, Capacitor_SMD:C_0402_1005Metric, F.Cu at (68.4, 182.2)
- added C82: 100nF, Capacitor_SMD:C_0805_2012Metric, F.Cu at (178.5, 109.4)
- added C95: 10nF, Capacitor_SMD:C_0603_1608Metric, F.Cu at (95.2, 104.0)
- added C96: 10nF, Capacitor_SMD:C_0603_1608Metric, F.Cu at (150.1, 104.0)
- added C97: 10nF, Capacitor_SMD:C_0603_1608Metric, F.Cu at (210.1, 94.8)
- added D10: SS34, Diode_SMD:D_SMA, F.Cu at (190.3, 150.7)
- added D11: SS34, Diode_SMD:D_SMA, F.Cu at (214.2, 150.6)
- added D12: SS34, Diode_SMD:D_SMA, F.Cu at (190.3, 130.2)
- added D13: SS34, Diode_SMD:D_SMA, F.Cu at (214.1, 130.2)
- added D2: SS34, Diode_SMD:D_SMA, F.Cu at (80.7, 150.7)
- added D3: SS34, Diode_SMD:D_SMA, F.Cu at (104.6, 150.7)
- added D4: SS34, Diode_SMD:D_SMA, F.Cu at (80.8, 130.3)
- added D5: SS34, Diode_SMD:D_SMA, F.Cu at (104.5, 130.3)
- added D6: SS34, Diode_SMD:D_SMA, F.Cu at (135.6, 150.7)
- added D7: SS34, Diode_SMD:D_SMA, F.Cu at (159.4, 150.6)
- added D8: SS34, Diode_SMD:D_SMA, F.Cu at (135.6, 130.2)
- added D9: SS34, Diode_SMD:D_SMA, F.Cu at (159.4, 130.2)
- added J1: Conn_02x06_Odd_Even, Connector_PinHeader_2.54mm:PinHeader_2x06_P2.54mm_Vertical, F.Cu at (-51.8, 89.0)
- added J10: Screw_Terminal_01x01, Bvrny's_library:M8_NutTerminal, F.Cu at (162.8, 55.0)
- added J11: Conn_02x02_Odd_Even, Connector_PinHeader_2.54mm:PinHeader_2x02_P2.54mm_Vertical, F.Cu at (142.0, 149.4)
- added J12: Conn_01x04_Pin, Connector_PinHeader_2.54mm:PinHeader_1x04_P2.54mm_Vertical, F.Cu at (156.0, 159.3)
- added J2: Conn_01x06_Pin, Connector_PinHeader_2.54mm:PinHeader_1x06_P2.54mm_Vertical, F.Cu at (160.2, 103.5)
- added J3: Conn_02x06_Odd_Even, Connector_PinHeader_2.54mm:PinHeader_2x06_P2.54mm_Vertical, F.Cu at (-37.5, 89.0)
- added J4: Screw_Terminal_01x01, Bvrny's_library:M8_NutTerminal, F.Cu at (70.2, 102.3)
- added J5: Screw_Terminal_01x01, Bvrny's_library:M8_NutTerminal, F.Cu at (125.0, 102.2)
- added J6: Screw_Terminal_01x01, Bvrny's_library:M8_NutTerminal, F.Cu at (179.8, 101.5)
- added J7: Conn_02x02_Odd_Even, Connector_PinHeader_2.54mm:PinHeader_2x02_P2.54mm_Vertical, F.Cu at (-51.8, 106.3)
- added J8: Conn_02x02_Odd_Even, Connector_PinHeader_2.54mm:PinHeader_2x02_P2.54mm_Vertical, F.Cu at (-51.8, 113.5)
- added J9: Screw_Terminal_01x01, Bvrny's_library:M8_NutTerminal, F.Cu at (100.4, 54.8)
- added Q10: IPT015N10N5, Package_TO_SOT_SMD:Infineon_PG-HSOF-8-1_ThermalVias, F.Cu at (182.8, 141.8)
- added Q11: IPT015N10N5, Package_TO_SOT_SMD:Infineon_PG-HSOF-8-1_ThermalVias, F.Cu at (206.7, 141.8)
- added Q12: IPT015N10N5, Package_TO_SOT_SMD:Infineon_PG-HSOF-8-1_ThermalVias, F.Cu at (182.8, 121.3)
- added Q13: IPT015N10N5, Package_TO_SOT_SMD:Infineon_PG-HSOF-8-1_ThermalVias, F.Cu at (206.7, 121.4)
- added Q18: BC860C, Package_TO_SOT_SMD:SOT-23, F.Cu at (87.6, 185.6)
- added Q19: BC860C, Package_TO_SOT_SMD:SOT-23, F.Cu at (45.2, 173.0)
- added Q2: IPT015N10N5, Package_TO_SOT_SMD:Infineon_PG-HSOF-8-1_ThermalVias, F.Cu at (73.2, 141.9)
- added Q20: BC860C, Package_TO_SOT_SMD:SOT-23, F.Cu at (65.4, 185.6)
- added Q3: IPT015N10N5, Package_TO_SOT_SMD:Infineon_PG-HSOF-8-1_ThermalVias, F.Cu at (97.1, 141.9)
- added Q4: IPT015N10N5, Package_TO_SOT_SMD:Infineon_PG-HSOF-8-1_ThermalVias, F.Cu at (73.2, 121.4)
- added Q5: IPT015N10N5, Package_TO_SOT_SMD:Infineon_PG-HSOF-8-1_ThermalVias, F.Cu at (97.1, 121.5)
- added Q6: IPT015N10N5, Package_TO_SOT_SMD:Infineon_PG-HSOF-8-1_ThermalVias, F.Cu at (128.1, 141.8)
- added Q7: IPT015N10N5, Package_TO_SOT_SMD:Infineon_PG-HSOF-8-1_ThermalVias, F.Cu at (151.9, 141.8)
- added Q8: IPT015N10N5, Package_TO_SOT_SMD:Infineon_PG-HSOF-8-1_ThermalVias, F.Cu at (128.1, 121.3)
- added Q9: IPT015N10N5, Package_TO_SOT_SMD:Infineon_PG-HSOF-8-1_ThermalVias, F.Cu at (151.9, 121.4)
- added R1: 100R, Resistor_SMD:R_0603_1608Metric, F.Cu at (97.6, 158.9)
- added R10: 51k, Resistor_SMD:R_0805_2012Metric, F.Cu at (91.3, 94.4)
- added R11: 51k, Resistor_SMD:R_0805_2012Metric, F.Cu at (93.3, 94.4)
- added R12: 4k7, Resistor_SMD:R_0805_2012Metric, F.Cu at (95.2, 94.4)
- added R13: 1R, Resistor_SMD:R_1206_3216Metric, F.Cu at (77.8, 133.7)
- added R14: 1R, Resistor_SMD:R_1206_3216Metric, F.Cu at (101.6, 133.7)
- added R15: 3R3, Resistor_SMD:R_1206_3216Metric, F.Cu at (77.8, 154.2)
- added R16: 3R3, Resistor_SMD:R_1206_3216Metric, F.Cu at (101.6, 129.1)
- added R17: 100R, Resistor_SMD:R_0603_1608Metric, F.Cu at (96.2, 89.3)
- added R18: 10k, Resistor_SMD:R_1206_3216Metric, F.Cu at (81.4, 124.4)
- added R19: 10k, Resistor_SMD:R_1206_3216Metric, F.Cu at (105.2, 124.5)
- added R2: 100R, Resistor_SMD:R_0603_1608Metric, F.Cu at (97.6, 157.3)
- added R20: 0.1mR, Bvrny's_library:R5930, F.Cu at (85.1, 113.5)
- added R21: 2K2, Resistor_SMD:R_0603_1608Metric, F.Cu at (88.1, 183.1)
- added R22: 560R, Resistor_SMD:R_0603_1608Metric, F.Cu at (91.1, 185.0)
- added R23: 0R, Resistor_SMD:R_0603_1608Metric, F.Cu at (88.1, 188.1)
- added R24: 100R, Resistor_SMD:R_0603_1608Metric, F.Cu at (152.6, 158.8)
- added R25: 10K, Resistor_SMD:R_0603_1608Metric, F.Cu at (91.1, 183.5)
- added R26: 100R, Resistor_SMD:R_0603_1608Metric, F.Cu at (152.6, 157.3)
- added R27: 100R, Resistor_SMD:R_0603_1608Metric, F.Cu at (155.3, 102.4)
- added R28: 1R, Resistor_SMD:R_1206_3216Metric, F.Cu at (132.6, 154.1)
- added R29: 1R, Resistor_SMD:R_1206_3216Metric, F.Cu at (156.5, 154.1)
- added R3: 100R, palmkiLib:R_0603_1608Metric, F.Cu at (100.5, 102.4)
- added R30: 3R3, Resistor_SMD:R_1206_3216Metric, F.Cu at (132.6, 149.4)
- added R31: 3R3, Resistor_SMD:R_1206_3216Metric, F.Cu at (156.5, 149.4)
- added R32: 10k, Resistor_SMD:R_1206_3216Metric, F.Cu at (136.2, 144.8)
- added R33: 10k, Resistor_SMD:R_1206_3216Metric, F.Cu at (160.0, 144.8)
- added R34: 51k, Resistor_SMD:R_0805_2012Metric, F.Cu at (146.1, 94.4)
- added R35: 51k, Resistor_SMD:R_0805_2012Metric, F.Cu at (148.1, 94.4)
- added R36: 4k7, Resistor_SMD:R_0805_2012Metric, F.Cu at (150.0, 94.4)
- added R37: 1R, Resistor_SMD:R_1206_3216Metric, F.Cu at (132.6, 133.6)
- added R38: 1R, Resistor_SMD:R_1206_3216Metric, F.Cu at (156.4, 133.6)
- added R39: 3R3, Resistor_SMD:R_1206_3216Metric, F.Cu at (132.6, 129.0)
- added R4: 1R, Resistor_SMD:R_1206_3216Metric, F.Cu at (77.8, 154.2)
- added R40: 3R3, Resistor_SMD:R_1206_3216Metric, F.Cu at (156.4, 129.0)
- added R41: 10k, Resistor_SMD:R_1206_3216Metric, F.Cu at (136.2, 124.3)
- added R42: 10k, Resistor_SMD:R_1206_3216Metric, F.Cu at (160.0, 124.4)
- added R43: 100R, Resistor_SMD:R_0603_1608Metric, F.Cu at (151.0, 89.2)
- added R44: 0.1mR, Bvrny's_library:R5930, F.Cu at (139.9, 113.4)
- added R45: 2K2, Resistor_SMD:R_0603_1608Metric, F.Cu at (45.6, 170.5)
- added R46: 560R, Resistor_SMD:R_0603_1608Metric, F.Cu at (48.7, 172.4)
- added R47: 0R, Resistor_SMD:R_0603_1608Metric, F.Cu at (45.6, 175.5)
- added R48: 10K, Resistor_SMD:R_0603_1608Metric, F.Cu at (48.7, 170.9)
- added R49: 100R, Resistor_SMD:R_0603_1608Metric, F.Cu at (207.2, 158.8)
- added R5: 1R, Resistor_SMD:R_1206_3216Metric, F.Cu at (101.6, 154.2)
- added R50: 100R, Resistor_SMD:R_0603_1608Metric, F.Cu at (207.2, 157.3)
- added R51: 100R, palmkiLib:R_0603_1608Metric, F.Cu at (210.2, 102.4)
- added R52: 1R, Resistor_SMD:R_1206_3216Metric, F.Cu at (187.4, 154.1)
- added R53: 1R, Resistor_SMD:R_1206_3216Metric, F.Cu at (211.2, 154.1)
- added R54: 3R3, Resistor_SMD:R_1206_3216Metric, F.Cu at (187.4, 149.4)
- added R55: 3R3, Resistor_SMD:R_1206_3216Metric, F.Cu at (211.2, 149.4)
- added R56: 10k, Resistor_SMD:R_1206_3216Metric, F.Cu at (190.9, 144.8)
- added R57: 10k, Resistor_SMD:R_1206_3216Metric, F.Cu at (214.8, 144.8)
- added R58: 51k, Resistor_SMD:R_0805_2012Metric, F.Cu at (201.0, 94.4)
- added R59: 51k, Resistor_SMD:R_0805_2012Metric, F.Cu at (203.0, 94.4)
- added R6: 3R3, Resistor_SMD:R_1206_3216Metric, F.Cu at (77.8, 149.5)
- added R60: 4k7, Resistor_SMD:R_0805_2012Metric, F.Cu at (204.9, 94.4)
- added R61: 1R, Resistor_SMD:R_1206_3216Metric, F.Cu at (187.4, 133.6)
- added R62: 1R, Resistor_SMD:R_1206_3216Metric, F.Cu at (211.2, 133.6)
- added R63: 3R3, Resistor_SMD:R_1206_3216Metric, F.Cu at (187.4, 128.9)
- added R64: 3R3, Resistor_SMD:R_1206_3216Metric, F.Cu at (211.2, 129.0)
- added R65: 10k, Resistor_SMD:R_1206_3216Metric, F.Cu at (191.0, 124.3)
- added R66: 10k, Resistor_SMD:R_1206_3216Metric, F.Cu at (214.7, 124.4)
- added R67: 100R, Resistor_SMD:R_0603_1608Metric, F.Cu at (205.9, 89.2)
- added R68: 0.1mR, Bvrny's_library:R5930, F.Cu at (194.7, 113.4)
- added R69: 2K2, Resistor_SMD:R_0603_1608Metric, F.Cu at (65.8, 183.1)
- added R7: 3R3, Resistor_SMD:R_1206_3216Metric, F.Cu at (101.6, 149.5)
- added R70: 560R, Resistor_SMD:R_0603_1608Metric, F.Cu at (68.9, 185.0)
- added R71: 0R, Resistor_SMD:R_0603_1608Metric, F.Cu at (65.9, 188.1)
- added R72: 10K, Resistor_SMD:R_0603_1608Metric, F.Cu at (68.9, 183.5)
- added R76: 10R, Resistor_SMD:R_0805_2012Metric, F.Cu at (96.2, 106.5)
- added R77: 10R, Resistor_SMD:R_0805_2012Metric, F.Cu at (98.2, 106.5)
- added R78: 10R, Resistor_SMD:R_0805_2012Metric, F.Cu at (94.3, 106.5)
- added R79: 10R, Resistor_SMD:R_0805_2012Metric, F.Cu at (92.3, 106.5)
- added R8: 10k, Resistor_SMD:R_1206_3216Metric, F.Cu at (81.3, 144.9)
- added R80: 10R, Resistor_SMD:R_0805_2012Metric, F.Cu at (151.0, 106.4)
- added R81: 10R, Resistor_SMD:R_0805_2012Metric, F.Cu at (153.0, 106.4)
- added R82: 10R, Resistor_SMD:R_0805_2012Metric, F.Cu at (147.1, 106.4)
- added R83: 10R, Resistor_SMD:R_0805_2012Metric, F.Cu at (149.1, 106.4)
- added R84: 10R, Resistor_SMD:R_0805_2012Metric, F.Cu at (207.6, 105.0)
- added R85: 10R, Resistor_SMD:R_0805_2012Metric, F.Cu at (205.7, 105.0)
- added R86: 10R, Resistor_SMD:R_0805_2012Metric, F.Cu at (203.7, 105.0)
- added R87: 10R, Resistor_SMD:R_0805_2012Metric, F.Cu at (201.7, 105.0)
- added R9: 10k, Resistor_SMD:R_1206_3216Metric, F.Cu at (105.2, 144.9)
- added R90: R, Resistor_SMD:R_1218_3246Metric, F.Cu at (99.3, 113.5)
- added R91: R, Resistor_SMD:R_1218_3246Metric, F.Cu at (154.2, 113.4)
- added R92: R, Resistor_SMD:R_1218_3246Metric, F.Cu at (208.9, 113.4)
- added R93: 18k, Resistor_SMD:R_0603_1608Metric, F.Cu at (91.1, 188.1)
- added R94: 18k, Resistor_SMD:R_0603_1608Metric, F.Cu at (48.7, 175.5)
- added R95: 18k, Resistor_SMD:R_0603_1608Metric, F.Cu at (68.9, 188.1)
- added TH1: NCP18XH103F03RB, Resistor_SMD:R_0603_1608Metric, F.Cu at (91.2, 186.5)
- added TH2: NCP18XH103F03RB, Resistor_SMD:R_0603_1608Metric, F.Cu at (48.7, 173.9)
- added TH3: NCP18XH103F03RB, Resistor_SMD:R_0603_1608Metric, F.Cu at (68.9, 186.6)
- added U10: TLV9001, Package_TO_SOT_SMD:SOT-23-5, F.Cu at (202.6, 90.6)
- added U2: INA240A2DR, Package_SO:SOIC-8_3.9x4.9mm_P1.27mm, F.Cu at (95.2, 100.5)
- added U3: UCC27211AQDDARQ1, Package_SO:SOIC-8-1EP_3.9x4.9mm_P1.27mm_EP2.95x4.9mm_Mask2.34x2.34mm_ThermalVias, F.Cu at (92.4, 156.8)
- added U4: TLV9001, Package_TO_SOT_SMD:SOT-23-5, F.Cu at (92.9, 90.6)
- added U5: UCC27211AQDDARQ1, Package_SO:SOIC-8-1EP_3.9x4.9mm_P1.27mm_EP2.95x4.9mm_Mask2.34x2.34mm_ThermalVias, F.Cu at (147.2, 156.7)
- added U6: INA240A2DR, Package_SO:SOIC-8_3.9x4.9mm_P1.27mm, F.Cu at (150.0, 100.5)
- added U7: TLV9001, Package_TO_SOT_SMD:SOT-23-5, F.Cu at (147.8, 90.6)
- added U8: UCC27211AQDDARQ1, Package_SO:SOIC-8-1EP_3.9x4.9mm_P1.27mm_EP2.95x4.9mm_Mask2.34x2.34mm_ThermalVias, F.Cu at (202.0, 156.8)
- added U9: INA240A2DR, Package_SO:SOIC-8_3.9x4.9mm_P1.27mm, F.Cu at (204.9, 100.5)
Routing:
- net +3.3VA: track 0.00 -> 47.7 mm, vias 0 -> 3
- net /Project Architecture/Phase V/HSgate: track 0.00 -> 42.1 mm
- net /Project Architecture/Phase V/LSgate: track 0.00 -> 29.1 mm
- net /Project Architecture/Phase V/phV_Shunt+: track 0.00 -> 20.7 mm
- net /Project Architecture/Phase V/phV_Shunt-: track 0.00 -> 19.3 mm
- net /Project Architecture/Phase V/phV_voltage: track 0.00 -> 9.48 mm
- net Net-(U5-HB): track 0.00 -> 9.39 mm, vias 0 -> 2
- net /Project Architecture/Phase V/phV_LO: track 0.00 -> 8.99 mm
- net /Project Architecture/Phase V/phV_current: track 0.00 -> 6.77 mm
- net Net-(U6-IN-): track 0.00 -> 6.70 mm
- net Net-(U6-IN+): track 0.00 -> 6.69 mm
- net Net-(U7-IN-): track 0.00 -> 5.78 mm, vias 0 -> 2
- net Net-(D6-K): track 0.00 -> 5.47 mm
- net Net-(D7-K): track 0.00 -> 5.22 mm
- net Net-(D9-K): track 0.00 -> 5.18 mm
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- added copper zone on F.Cu, net +12V
- added copper zone on B.Cu, net +VSYS
- added copper zone on F.Cu, net +VSYS
- added copper zone on B.Cu, net /Project Architecture/Phase U/PhaseU_out
- added copper zone on F.Cu, net /Project Architecture/Phase U/PhaseU_out
- added copper zone on F.Cu, net /Project Architecture/Phase V/HSgate
- added copper zone on F.Cu, net /Project Architecture/Phase V/LSgate
- added copper zone on B.Cu, net /Project Architecture/Phase V/PhaseV_out
- added copper zone on F.Cu, net /Project Architecture/Phase V/PhaseV_out
- added copper zone on F.Cu, net /Project Architecture/Phase V/phV_Shunt+
- added copper zone on F.Cu, net /Project Architecture/Phase V/phV_Shunt-
- added copper zone on F.Cu, net /Project Architecture/Phase V/phV_current
- added copper zone on F.Cu, net /Project Architecture/Phase V/phV_voltage
- added copper zone on B.Cu, net /Project Architecture/Phase W/PhaseW_out
- added copper zone on F.Cu, net /Project Architecture/Phase W/PhaseW_out
- added copper zone on B.Cu, net GND
- added copper zone on F.Cu, net GND
- added copper zone on F.Cu, net Net-(C105-Pad1)
- added copper zone on F.Cu, net Net-(D6-A)
- added copper zone on F.Cu, net Net-(D7-A)
- added copper zone on F.Cu, net Net-(D8-A)
- added copper zone on F.Cu, net Net-(D9-A)
- added copper zone on B.Cu, net Net-(U3-HS)
- added copper zone on F.Cu, net Net-(U3-HS)
- added copper zone on B.Cu, net Net-(U5-HS)
- added copper zone on F.Cu, net Net-(U5-HS)
- added copper zone on F.Cu, net Net-(U6-IN+)
- added copper zone on F.Cu, net Net-(U6-IN-)
- added copper zone on F.Cu, net Net-(U7-IN+)
- added copper zone on B.Cu, net Net-(U8-HS)
- added copper zone on F.Cu, net Net-(U8-HS)
Other:
- board outline added: 160 x 110 mm

Commit message: Moved the current and voltage sensing OpAmp's to Vector
Parts:
- removed C29, C30, C38, C40, C44, C49, C56, C58, C66, C68, C74, C76: 100nF, Capacitor_SMD:C_0402_1005Metric
- removed C36, C55, C73: 2.2nF, Capacitor_SMD:C_0603_1608Metric
- removed C39, C57, C75: 3.3nF, Capacitor_SMD:C_0603_1608Metric
- removed C41, C59, C77: 1nF, Capacitor_SMD:C_0603_1608Metric
- removed C95, C96, C97: 10nF, Capacitor_SMD:C_0603_1608Metric
- removed R10, R11, R34, R35, R58, R59: 51k, Resistor_SMD:R_0805_2012Metric
- removed R12, R36, R60: 4k7, Resistor_SMD:R_0805_2012Metric
- removed R17, R27, R43, R67: 100R, Resistor_SMD:R_0603_1608Metric
- removed R3, R51: 100R, palmkiLib:R_0603_1608Metric
- removed U10, U4, U7: TLV9001, Package_TO_SOT_SMD:SOT-23-5
- removed U2, U6, U9: INA240A2DR, Package_SO:SOIC-8_3.9x4.9mm_P1.27mm
- added C100: 10nF, Capacitor_SMD:C_0603_1608Metric, F.Cu at (157.6, 87.3)
- added C101: 10nF, Capacitor_SMD:C_0603_1608Metric, F.Cu at (211.0, 86.4)
- added C99: 10nF, Capacitor_SMD:C_0603_1608Metric, F.Cu at (49.0, 88.3)
- moved C61 209.8 mm to (326.6, 75.1), turned to 0 degrees
- moved C60 207.5 mm to (326.6, 77.1), turned to 0 degrees
- moved C62 205.2 mm to (326.6, 79.1), turned to 0 degrees
- moved C140 198.9 mm to (320.9, 66.3), turned to -90 degrees
- moved C125 196.5 mm to (317.7, 66.3), turned to -90 degrees
- moved C109 91.6 mm to (246.4, -19.6)
- moved C118 91.6 mm to (185.1, -19.7)
- moved C108 91.6 mm to (227.8, -19.6)
- moved C120 91.6 mm to (104.9, -19.6)
- moved C122 91.6 mm to (123.5, -19.6)
- moved C124 91.6 mm to (166.5, -19.7)
- moved J9 89.4 mm to (120.1, 142.0), turned to -90 degrees
- moved J2 88.1 mm to (146.0, 190.5)
- moved R91 81.3 mm to (127.9, 190.4)
- moved C105 74.6 mm to (129.7, 183.2)
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Connections:
- net Net-(U2-IN+) renamed /Project Architecture/Phase U/phU_I-
- net Net-(U2-IN-) renamed /Project Architecture/Phase U/phU_I+
- net Net-(U6-IN+) renamed /Project Architecture/Phase V/phV_I+
- net Net-(U6-IN-) renamed /Project Architecture/Phase V/phV_I-
- net Net-(U9-IN-) renamed /Project Architecture/Phase W/phW_I-
- J1 pad 12: /Project Architecture/Phase U/phU_voltage -> unconnected-(J1-Pin_12-Pad12)
- J1 pad 4: /Project Architecture/Phase U/phU_NTCctrl -> unconnected-(J1-Pin_4-Pad4)
- J1 pad 8: /Project Architecture/Phase U/phU_NTCout -> unconnected-(J1-Pin_8-Pad8)
- J1 pad 9: /Project Architecture/Phase U/phU_current -> unconnected-(J1-Pin_9-Pad9)
- J2 pad 3: /Project Architecture/Phase V/phV_current -> unconnected-(J2-Pin_3-Pad3)
- J2 pad 5: /Project Architecture/Phase V/phV_voltage -> unconnected-(J2-Pin_5-Pad5)
- J3 pad 12: /Project Architecture/Phase W/phW_voltage -> /Project Architecture/phW_voltage
- J3 pad 9: /Project Architecture/Phase W/phW_current -> /Project Architecture/Phase W/phW_I+
- R68 pad 2: /Project Architecture/Phase W/phU_Shunt+ -> /Project Architecture/Phase W/phW_Shunt+
- R68 pad 3: /Project Architecture/Phase W/phU_Shunt- -> /Project Architecture/Phase W/phW_Shunt-
- R76 pad 1: /Project Architecture/Phase U/phU_Shunt+ -> /Project Architecture/Phase U/phU_Shunt-
- R77 pad 1: /Project Architecture/Phase U/phU_Shunt+ -> /Project Architecture/Phase U/phU_Shunt-
- R78 pad 1: /Project Architecture/Phase U/phU_Shunt- -> /Project Architecture/Phase U/phU_Shunt+
- R79 pad 1: /Project Architecture/Phase U/phU_Shunt- -> /Project Architecture/Phase U/phU_Shunt+
- R84 pad 2: Net-(U9-IN+) -> /Project Architecture/Phase W/phW_I+
- R85 pad 2: Net-(U9-IN+) -> /Project Architecture/Phase W/phW_I+
Routing:
- net +3.3VA: track 47.7 -> 7.31 mm, vias 3 -> 0
- net /Project Architecture/Phase V/phV_voltage: track 9.48 -> 0.00 mm
- net Net-(U5-HB): track 9.39 -> 2.44 mm, vias 2 -> 0
- net /Project Architecture/Phase V/phV_current: track 6.77 -> 0.00 mm
- net /Project Architecture/Phase V/phV_I-: track 6.70 -> 0.00 mm
- net /Project Architecture/Phase V/phV_I+: track 6.69 -> 0.00 mm
- net /Project Architecture/Phase V/phV_Shunt+: track 20.7 -> 14.7 mm
- net Net-(U7-IN-): track 5.78 -> 0.00 mm, vias 2 -> 0
- net Net-(D13-K): track 0.00 -> 5.33 mm
- net Net-(D3-K): track 0.00 -> 5.33 mm
- net Net-(D10-K): track 0.00 -> 5.29 mm
- net Net-(D4-K): track 0.00 -> 5.25 mm
- net Net-(D2-K): track 0.00 -> 5.24 mm
- net Net-(D11-K): track 0.00 -> 5.20 mm
- net Net-(D12-K): track 0.00 -> 5.13 mm
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- added copper zone on F.Cu, net (none)
- added copper zone on F.Cu, net /Project Architecture/Phase U/HSgate
- added copper zone on F.Cu, net /Project Architecture/Phase U/LSgate
- added copper zone on F.Cu, net /Project Architecture/Phase W/HSgate
- added copper zone on F.Cu, net /Project Architecture/Phase W/LSgate
- added copper zone on F.Cu, net Net-(D10-A)
- added copper zone on F.Cu, net Net-(D11-A)
- added copper zone on F.Cu, net Net-(D12-A)
- added copper zone on F.Cu, net Net-(D13-A)
- added copper zone on F.Cu, net Net-(D2-A)
- added copper zone on F.Cu, net Net-(D3-A)
- added copper zone on F.Cu, net Net-(D4-A)
- added copper zone on F.Cu, net Net-(D5-A)
- removed copper zone on F.Cu, net /Project Architecture/Phase V/phV_I+
- removed copper zone on F.Cu, net /Project Architecture/Phase V/phV_I-
- removed copper zone on F.Cu, net /Project Architecture/Phase V/phV_current
- removed copper zone on F.Cu, net /Project Architecture/Phase V/phV_voltage
- removed copper zone on F.Cu, net Net-(C105-Pad1)
- removed copper zone on F.Cu, net Net-(U7-IN+)

Commit message: Changed Flux layout so be top to bottom
Parts:
- moved R82 158.3 mm to (298.4, 151.5), turned to -90 degrees
- moved C53 157.8 mm to (272.8, 45.6), turned to 90 degrees
- moved C54 157.2 mm to (269.7, 45.5), turned to 180 degrees
- moved C142 156.8 mm to (260.5, 44.4), turned to 180 degrees
- moved R83 155.6 mm to (296.4, 151.5), turned to -90 degrees
- moved C46 154.0 mm to (276.6, 49.3), turned to -90 degrees
- moved C128 154.0 mm to (260.5, 46.4), turned to 180 degrees
- moved C42 153.2 mm to (274.2, 49.3), turned to -90 degrees
- moved C100 153.1 mm to (295.5, 154.0), turned to 180 degrees
- moved R80 153.0 mm to (294.5, 151.5), turned to -90 degrees
- moved C64 151.1 mm to (260.5, 48.4), turned to 180 degrees
- moved U5 150.5 mm to (270.3, 50.4), turned to -90 degrees
- moved C125 150.5 mm to (238.4, 194.3)
- moved C140 150.5 mm to (241.7, 194.3)
- moved C62 150.5 mm to (247.4, 207.0)
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Routing:
- net /Project Architecture/Phase V/HSgate: track 42.6 -> 8.84 mm
- net Net-(D5-A): track 0.00 -> 20.4 mm
- net Net-(D9-A): track 0.00 -> 20.4 mm
- net /Project Architecture/Phase V/LSgate: track 29.1 -> 9.06 mm
- net Net-(D4-A): track 0.00 -> 18.0 mm
- net Net-(D8-A): track 0.00 -> 17.9 mm
- net /Project Architecture/Phase U/phU_Shunt+: track 0.00 -> 14.0 mm
- net /Project Architecture/Phase U/phU_Shunt-: track 0.00 -> 13.6 mm
- net /Project Architecture/Phase V/phV_Shunt+: track 14.7 -> 1.42 mm
- net /Project Architecture/Phase V/phV_Shunt-: track 14.9 -> 2.04 mm
- net Net-(D3-A): track 0.00 -> 11.8 mm
- net Net-(D7-A): track 0.00 -> 11.7 mm
- net /Project Architecture/Phase V/phV_LO: track 8.99 -> 0.00 mm
- net Net-(D2-A): track 0.00 -> 8.76 mm
- net Net-(D6-A): track 0.00 -> 8.65 mm
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- removed copper zone on B.Cu, net +VSYS
- removed copper zone on F.Cu, net +VSYS
- removed copper zone on F.Cu, net /Project Architecture/Phase U/HSgate
- removed copper zone on F.Cu, net /Project Architecture/Phase U/LSgate
- removed copper zone on F.Cu, net /Project Architecture/Phase V/HSgate
- removed copper zone on F.Cu, net /Project Architecture/Phase V/LSgate
- removed copper zone on F.Cu, net /Project Architecture/Phase W/HSgate
- removed copper zone on F.Cu, net /Project Architecture/Phase W/LSgate
- removed copper zone on B.Cu, net /Project Architecture/Phase W/PhaseW_out
- removed copper zone on F.Cu, net /Project Architecture/Phase W/PhaseW_out
- removed copper zone on F.Cu, net Net-(D10-A)
- removed copper zone on F.Cu, net Net-(D11-A)
- removed copper zone on F.Cu, net Net-(D12-A)
- removed copper zone on F.Cu, net Net-(D13-A)
- removed copper zone on F.Cu, net Net-(D2-A)
- removed copper zone on F.Cu, net Net-(D3-A)
- removed copper zone on F.Cu, net Net-(D4-A)
- removed copper zone on F.Cu, net Net-(D5-A)
- removed copper zone on F.Cu, net Net-(D6-A)
- removed copper zone on F.Cu, net Net-(D7-A)
- removed copper zone on F.Cu, net Net-(D8-A)
- removed copper zone on F.Cu, net Net-(D9-A)
Other:
- board size 160 x 110 mm -> 160 x 100 mm
