File: PCBA-FLUX-01A/PCBA-FLUX-01A.kicad_pcb (KiCad board)
At the start: 2 copper layers, 160 x 100 mm, 164 parts, among them J10 Screw_Terminal_01x01, J4 Screw_Terminal_01x01, J5 Screw_Terminal_01x01, J6 Screw_Terminal_01x01, J7 Conn_02x02_Odd_Even, J8 Conn_02x02_Odd_Even, J9 Screw_Terminal_01x01, Q10 IPT015N10N5, Q11 IPT015N10N5, Q12 IPT015N10N5, Q13 IPT015N10N5, Q18 BC860C, Q19 BC860C, Q2 IPT015N10N5, Q20 BC860C, Q3 IPT015N10N5, Q4 IPT015N10N5, Q5 IPT015N10N5, Q6 IPT015N10N5, Q7 IPT015N10N5, Q8 IPT015N10N5, Q9 IPT015N10N5

Commit message: :|
Parts:
- removed the REF** at (114.7, 108.9)
- added REF**: PinHeader_2x05_P2.54mm_Vertical, Connector_PinHeader_2.54mm:PinHeader_2x05_P2.54mm_Vertical, F.Cu at (188.7, 72.7)
- added REF**: PinHeader_2x05_P2.54mm_Vertical, Connector_PinHeader_2.54mm:PinHeader_2x05_P2.54mm_Vertical, F.Cu at (134.6, 72.7)
- added REF**: PinHeader_2x05_P2.54mm_Vertical, Connector_PinHeader_2.54mm:PinHeader_2x05_P2.54mm_Vertical, F.Cu at (94.3, 91.4)
- added REF**: PinHeader_2x05_P2.54mm_Vertical, Connector_PinHeader_2.54mm:PinHeader_2x05_P2.54mm_Vertical, F.Cu at (242.5, 107.1)
- added REF**: PinHeader_2x05_P2.54mm_Vertical, Connector_PinHeader_2.54mm:PinHeader_2x05_P2.54mm_Vertical, F.Cu at (243.1, 71.8)
- added REF**: PinHeader_2x05_P2.54mm_Vertical, Connector_PinHeader_2.54mm:PinHeader_2x05_P2.54mm_Vertical, F.Cu at (188.5, 107.3)
- added REF**: PinHeader_2x05_P2.54mm_Vertical, Connector_PinHeader_2.54mm:PinHeader_2x05_P2.54mm_Vertical, F.Cu at (134.3, 107.2)
- moved C80 236.5 mm to (38.6, 137.1)
- moved C82 236.5 mm to (38.6, 139.1)
- moved C139 228.3 mm to (40.0, 148.5)
- moved C78 228.3 mm to (40.0, 144.5)
- moved C79 228.3 mm to (40.0, 146.5)
- moved C140 228.3 mm to (16.8, 154.8)
- moved C60 228.3 mm to (22.5, 165.6)
- moved C61 228.3 mm to (22.5, 163.5)
- moved C62 228.3 mm to (22.5, 167.6)
- moved C125 228.3 mm to (13.6, 154.8)
- moved C154 213.7 mm to (274.4, 5.67), turned to 0 degrees
- moved C112 178.1 mm to (249.6, 156.8)
- moved C113 178.1 mm to (252.8, 156.8)
- moved C116 178.1 mm to (262.6, 156.8)
- moved C114 178.1 mm to (256.1, 156.8)
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Routing:
- net Net-(D5-A): track 15.6 -> 0.00 mm
- net /Project Architecture/Phase U/phU_Shunt+: track 14.0 -> 0.00 mm
- net /Project Architecture/Phase U/phU_Shunt-: track 13.6 -> 0.00 mm
- net Net-(D9-A): track 15.7 -> 2.72 mm
- net Net-(D13-A): track 15.7 -> 2.79 mm
- net Net-(D11-K): track 8.16 -> 0.00 mm
- net Net-(D12-K): track 8.13 -> 0.00 mm
- net Net-(D7-K): track 8.13 -> 0.00 mm
- net Net-(D13-K): track 8.13 -> 0.00 mm
- net Net-(D8-K): track 8.12 -> 0.00 mm
- net Net-(D10-K): track 8.11 -> 0.00 mm
- net Net-(D9-K): track 7.93 -> 0.00 mm
- net Net-(D5-K): track 7.89 -> 0.00 mm
- net Net-(D3-K): track 7.81 -> 0.00 mm
- net Net-(D2-K): track 7.70 -> 0.00 mm
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- added copper zone on B.Cu, net /Project Architecture/Phase W/PhaseW_out
- added copper zone on F.Cu, net /Project Architecture/Phase W/PhaseW_out
- removed copper zone on F.Cu, net Net-(D10-A)
- removed copper zone on F.Cu, net Net-(D11-A)
- removed copper zone on F.Cu, net Net-(D12-A)
- removed copper zone on F.Cu, net Net-(D13-A)
- removed copper zone on F.Cu, net Net-(D2-A)
- removed copper zone on F.Cu, net Net-(D3-A)
- removed copper zone on F.Cu, net Net-(D4-A)
- removed copper zone on F.Cu, net Net-(D5-A)
- removed copper zone on F.Cu, net Net-(D6-A)
- removed copper zone on F.Cu, net Net-(D8-A)
- removed copper zone on F.Cu, net Net-(D9-A)
Other:
- board size 160 x 100 mm -> 185 x 100 mm

Commit message: :}
Parts:
- removed REF** (x7): PinHeader_2x05_P2.54mm_Vertical, Connector_PinHeader_2.54mm:PinHeader_2x05_P2.54mm_Vertical
- added J1: Conn_02x07_Odd_Even, Connector_PinHeader_2.54mm:PinHeader_2x07_P2.54mm_Vertical, F.Cu at (196.9, 110.3)
- added J11: Conn_02x02_Odd_Even, Connector_PinHeader_2.54mm:PinHeader_2x02_P2.54mm_Vertical, F.Cu at (100.6, 107.8)
- added J2: Conn_02x07_Odd_Even, Connector_PinHeader_2.54mm:PinHeader_2x07_P2.54mm_Vertical, F.Cu at (142.4, 110.3)
- added J3: Conn_02x06_Odd_Even, Connector_PinHeader_2.54mm:PinHeader_2x06_P2.54mm_Vertical, F.Cu at (251.5, 110.3)
- moved C101 232.9 mm to (253.9, 102.0), turned to -90 degrees
- moved R84 231.5 mm to (251.4, 105.0), turned to 0 degrees
- moved R85 230.3 mm to (251.4, 103.0), turned to 0 degrees
- moved R86 229.1 mm to (251.4, 101.1), turned to 0 degrees
- moved R87 228.0 mm to (251.4, 99.1), turned to 0 degrees
- moved J7 175.5 mm to (265.7, 42.3)
- moved J8 175.4 mm to (265.7, 132.6)
- moved R79 94.9 mm to (142.3, 102.9), turned to 0 degrees
- moved R76 94.1 mm to (142.3, 99.0), turned to 0 degrees
- moved C99 92.6 mm to (144.8, 102.0), turned to -90 degrees
- moved R78 92.2 mm to (142.3, 104.9), turned to 0 degrees
- moved R77 91.3 mm to (142.3, 101.0), turned to 0 degrees
- moved C100 50.3 mm to (199.3, 102.0), turned to -90 degrees
- moved R82 48.4 mm to (196.9, 99.0), turned to 0 degrees
- moved R83 47.4 mm to (196.9, 101.0), turned to 0 degrees
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Connections:
- C48 pad 1: /Project Architecture/Phase U/phU_NTCout -> /Project Architecture/Phase U/PhaseU_out
- J5 pad 1: /Project Architecture/Phase V/PhaseV_out -> unconnected-(J5-Pin_1-Pad1)
- J6 pad 1: /Project Architecture/Phase W/PhaseW_out -> unconnected-(J6-Pin_1-Pad1)
- R13 pad 1: /Project Architecture/Phase U/phU_HSgate2 -> /Project Architecture/Phase U/PhaseU_out
- R15 pad 1: /Project Architecture/Phase U/phU_HSgate2 -> /Project Architecture/Phase U/PhaseU_out
- R21 pad 1: /Project Architecture/Phase U/phU_NTCctrl -> /Project Architecture/Phase U/PhaseU_out
- R25 pad 2: /Project Architecture/Phase U/phU_NTCout -> /Project Architecture/Phase U/PhaseU_out
- R4 pad 1: /Project Architecture/Phase U/phU_HSgate1 -> /Project Architecture/Phase U/PhaseU_out
- R6 pad 1: /Project Architecture/Phase U/phU_HSgate1 -> /Project Architecture/Phase U/PhaseU_out
- R61 pad 1: /Project Architecture/Phase W/phW_HSgate2 -> /Project Architecture/Phase W/PhaseW_out
- R63 pad 1: /Project Architecture/Phase W/phW_HSgate2 -> /Project Architecture/Phase W/PhaseW_out
Routing:
- net /Project Architecture/Phase V/phV_Shunt+: track 1.42 -> 24.1 mm
- net /Project Architecture/Phase V/phV_HS: track 0.00 -> 22.5 mm
- net /Project Architecture/Phase V/phV_Shunt-: track 2.04 -> 23.4 mm
- net Net-(D4-A): track 18.0 -> 0.00 mm
- net Net-(D12-A): track 13.2 -> 0.00 mm
- net Net-(D6-A): track 9.14 -> 0.00 mm
- net Net-(D10-A): track 4.18 -> 0.00 mm
- net Net-(D2-A): track 4.08 -> 0.00 mm
- net /Project Architecture/Phase V/phV_LSgate2: track 2.32 -> 5.74 mm
- net Net-(D7-A): track 2.89 -> 0.00 mm
- net Net-(D13-A): track 2.79 -> 0.00 mm
- net Net-(D6-K): track 2.74 -> 0.00 mm
- net Net-(D4-K): track 2.73 -> 0.00 mm
- net Net-(D9-A): track 2.72 -> 0.00 mm
- net /Project Architecture/Phase W/phW_HSgate1: track 2.33 -> 0.00 mm
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- removed copper zone on B.Cu, net +VSYS
- removed copper zone on F.Cu, net +VSYS
- removed copper zone on B.Cu, net /Project Architecture/Phase W/phW_HS
- removed copper zone on F.Cu, net Net-(D7-A)
Other:
- board size 185 x 100 mm -> 190 x 100 mm

Commit message: :{
Parts:
- removed C112, C113, C114, C115, C116, C119, C121, C123, C125, C127, C140, C141: 10uF, Capacitor_SMD:C_1210_3225Metric
- removed C117, C128, C142, C43, C45, C47, C50, C60, C61, C62, C64: 100nF, Capacitor_SMD:C_0805_2012Metric
- removed NT1, NT2, NT3: NetTie_2, NetTie:NetTie-2_SMD_Pad0.5mm
- added C56: 3.3nF, Capacitor_SMD:C_0603_1608Metric, F.Cu at (120.3, 117.8)
- added C57: 3.3nF, Capacitor_SMD:C_0603_1608Metric, F.Cu at (174.9, 117.8)
- added C58: 3.3nF, Capacitor_SMD:C_0603_1608Metric, F.Cu at (229.5, 117.9)
- added J12: Conn_01x03_Pin, Connector_PinHeader_2.54mm:PinHeader_1x03_P2.54mm_Vertical, F.Cu at (128.4, 77.4)
- added J13: Conn_01x03_Pin, Connector_PinHeader_2.54mm:PinHeader_1x03_P2.54mm_Vertical, F.Cu at (167.7, 77.4)
- added J14: Conn_01x03_Pin, Connector_PinHeader_2.54mm:PinHeader_1x03_P2.54mm_Vertical, F.Cu at (128.5, 112.4)
- added J15: Conn_01x03_Pin, Connector_PinHeader_2.54mm:PinHeader_1x03_P2.54mm_Vertical, F.Cu at (167.8, 112.5)
- added J16: Conn_01x03_Pin, Connector_PinHeader_2.54mm:PinHeader_1x03_P2.54mm_Vertical, F.Cu at (183.1, 77.4)
- added J17: Conn_01x03_Pin, Connector_PinHeader_2.54mm:PinHeader_1x03_P2.54mm_Vertical, F.Cu at (222.3, 77.6)
- added J18: Conn_01x03_Pin, Connector_PinHeader_2.54mm:PinHeader_1x03_P2.54mm_Vertical, F.Cu at (183.1, 112.5)
- added J19: Conn_01x03_Pin, Connector_PinHeader_2.54mm:PinHeader_1x03_P2.54mm_Vertical, F.Cu at (222.4, 112.5)
- added J20: Conn_01x05_Pin, Connector_PinHeader_2.54mm:PinHeader_1x05_P2.54mm_Vertical, F.Cu at (232.1, 107.4)
- added J21: Conn_01x04_Pin, Connector_PinHeader_2.54mm:PinHeader_1x04_P2.54mm_Vertical, F.Cu at (231.0, 77.6)
- added J22: Conn_01x05_Pin, Connector_PinHeader_2.54mm:PinHeader_1x05_P2.54mm_Vertical, F.Cu at (177.5, 107.4)
- added J23: Conn_01x04_Pin, Connector_PinHeader_2.54mm:PinHeader_1x04_P2.54mm_Vertical, F.Cu at (177.4, 137.2)
- added J24: Conn_01x05_Pin, Connector_PinHeader_2.54mm:PinHeader_1x05_P2.54mm_Vertical, F.Cu at (122.9, 107.4)
- added J25: Conn_01x04_Pin, Connector_PinHeader_2.54mm:PinHeader_1x04_P2.54mm_Vertical, F.Cu at (33.2, 106.7)
- added R26: 51k, Resistor_SMD:R_0805_2012Metric, F.Cu at (125.7, 110.8)
- added R27: 51k, Resistor_SMD:R_0805_2012Metric, F.Cu at (125.7, 114.2)
- added R34: 4k7, Resistor_SMD:R_0805_2012Metric, F.Cu at (125.7, 117.6)
- added R35: 51k, Resistor_SMD:R_0805_2012Metric, F.Cu at (180.3, 110.8)
- added R36: 51k, Resistor_SMD:R_0805_2012Metric, F.Cu at (180.3, 114.2)
- added R43: 4k7, Resistor_SMD:R_0805_2012Metric, F.Cu at (180.3, 117.6)
- added R49: 51k, Resistor_SMD:R_0805_2012Metric, F.Cu at (234.9, 110.8)
- added R50: 51k, Resistor_SMD:R_0805_2012Metric, F.Cu at (234.9, 114.2)
- added R51: 4k7, Resistor_SMD:R_0805_2012Metric, F.Cu at (234.9, 117.7)
- added REF**: CP_Radial_D12.5mm_P5.00mm, Capacitor_THT:CP_Radial_D12.5mm_P5.00mm, F.Cu at (64.9, 51.6)
- added REF**: CP_Radial_D12.5mm_P5.00mm, Capacitor_THT:CP_Radial_D12.5mm_P5.00mm, F.Cu at (65.0, 64.8)
- added REF**: CP_Radial_D12.5mm_P5.00mm, Capacitor_THT:CP_Radial_D12.5mm_P5.00mm, F.Cu at (251.9, 51.6)
- added REF**: CP_Radial_D12.5mm_P5.00mm, Capacitor_THT:CP_Radial_D12.5mm_P5.00mm, F.Cu at (252.0, 103.8)
- added REF**: CP_Radial_D12.5mm_P5.00mm, Capacitor_THT:CP_Radial_D12.5mm_P5.00mm, F.Cu at (77.9, 51.6)
- added REF**: CP_Radial_D12.5mm_P5.00mm, Capacitor_THT:CP_Radial_D12.5mm_P5.00mm, F.Cu at (65.0, 104.0)
- added REF**: CP_Radial_D12.5mm_P5.00mm, Capacitor_THT:CP_Radial_D12.5mm_P5.00mm, F.Cu at (251.9, 64.6)
- added REF**: CP_Radial_D12.5mm_P5.00mm, Capacitor_THT:CP_Radial_D12.5mm_P5.00mm, F.Cu at (252.0, 130.0)
- added REF**: CP_Radial_D12.5mm_P5.00mm, Capacitor_THT:CP_Radial_D12.5mm_P5.00mm, F.Cu at (252.0, 116.9)
- added REF**: CP_Radial_D12.5mm_P5.00mm, Capacitor_THT:CP_Radial_D12.5mm_P5.00mm, F.Cu at (65.0, 130.1)
- added REF**: CP_Radial_D12.5mm_P5.00mm, Capacitor_THT:CP_Radial_D12.5mm_P5.00mm, F.Cu at (252.0, 90.7)
- added REF**: CP_Radial_D12.5mm_P5.00mm, Capacitor_THT:CP_Radial_D12.5mm_P5.00mm, F.Cu at (65.0, 77.9)
- added REF**: CP_Radial_D12.5mm_P5.00mm, Capacitor_THT:CP_Radial_D12.5mm_P5.00mm, F.Cu at (78.6, 134.1)
- added REF**: CP_Radial_D12.5mm_P5.00mm, Capacitor_THT:CP_Radial_D12.5mm_P5.00mm, F.Cu at (252.0, 77.7)
- added REF**: CP_Radial_D12.5mm_P5.00mm, Capacitor_THT:CP_Radial_D12.5mm_P5.00mm, F.Cu at (65.0, 117.0)
- added REF**: CP_Radial_D12.5mm_P5.00mm, Capacitor_THT:CP_Radial_D12.5mm_P5.00mm, F.Cu at (65.0, 90.9)
- J1, J2: value Conn_02x07_Odd_Even -> Conn_01x03_Pin; footprint Connector_PinHeader_2.54mm:PinHeader_2x07_P2.54mm_Vertical -> Connector_PinHeader_2.54mm:PinHeader_1x03_P2.54mm_Vertical
- J11: value Conn_02x02_Odd_Even -> Conn_01x03_Pin; footprint Connector_PinHeader_2.54mm:PinHeader_2x02_P2.54mm_Vertical -> Connector_PinHeader_2.54mm:PinHeader_1x03_P2.54mm_Vertical
- J3: value Conn_02x06_Odd_Even -> Conn_01x03_Pin; footprint Connector_PinHeader_2.54mm:PinHeader_2x06_P2.54mm_Vertical -> Connector_PinHeader_2.54mm:PinHeader_1x03_P2.54mm_Vertical
- moved R46 238.1 mm to (228.9, 28.4)
- moved R47 238.1 mm to (225.9, 31.4)
- moved R94 238.1 mm to (228.9, 31.4)
- moved TH2 238.1 mm to (228.9, 29.9)
- moved Q19 236.3 mm to (223.2, 28.9)
- moved R48 236.3 mm to (226.7, 26.9)
- moved C63 236.3 mm to (226.2, 25.6)
- moved R45 236.3 mm to (223.6, 26.4)
- moved R69 229.0 mm to (256.6, 73.2), turned to -90 degrees
- moved TH3 211.8 mm to (237.5, 72.2), turned to 0 degrees
- moved C139 211.5 mm to (166.8, -20.8)
- moved C78 211.5 mm to (166.8, -24.8)
- moved C79 211.5 mm to (166.8, -22.8)
- moved C80 211.5 mm to (165.4, -32.2)
- moved C82 211.5 mm to (165.4, -30.2)
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Connections:
- C48 pad 1: /Project Architecture/Phase U/PhaseU_out -> /Project Architecture/Phase U/phU_NTCout
- J1 pad 1: GND -> /Project Architecture/Phase U/phU_HSgate1
- J1 pad 2: /Project Architecture/Phase V/phV_LSgate2 -> GND
- J1 pad 3: /Project Architecture/Phase V/phV_HS -> /Project Architecture/Phase U/phU_HS
- J11 pad 1: GND -> /Project Architecture/Phase U/phU_HS
- J11 pad 2: /Project Architecture/Phase U/phU_LSgate1 -> GND
- J11 pad 3: /Project Architecture/Phase U/phU_HS -> /Project Architecture/Phase U/phU_LSgate2
- J2 pad 1: GND -> /Project Architecture/Phase U/phU_HSgate2
- J2 pad 2: /Project Architecture/Phase U/phU_LSgate2 -> GND
- J3 pad 1: GND -> /Project Architecture/Phase U/phU_HS
- J3 pad 2: /Project Architecture/Phase W/phW_LSgate2 -> GND
- J3 pad 3: /Project Architecture/Phase W/phW_HS -> /Project Architecture/Phase U/phU_LSgate1
- J4 pad 1: unconnected-(J4-Pin_1-Pad1) -> /Project Architecture/Phase U/PhaseU_out
- J5 pad 1: unconnected-(J5-Pin_1-Pad1) -> /Project Architecture/Phase V/PhaseV_out
- J6 pad 1: unconnected-(J6-Pin_1-Pad1) -> /Project Architecture/Phase W/PhaseW_out
- R13 pad 1: /Project Architecture/Phase U/PhaseU_out -> /Project Architecture/Phase U/phU_HSgate2
- R15 pad 1: /Project Architecture/Phase U/PhaseU_out -> /Project Architecture/Phase U/phU_HSgate2
- R21 pad 1: /Project Architecture/Phase U/PhaseU_out -> /Project Architecture/Phase U/phU_NTCctrl
- R25 pad 2: /Project Architecture/Phase U/PhaseU_out -> /Project Architecture/Phase U/phU_NTCout
- R4 pad 1: /Project Architecture/Phase U/PhaseU_out -> /Project Architecture/Phase U/phU_HSgate1
- R6 pad 1: /Project Architecture/Phase U/PhaseU_out -> /Project Architecture/Phase U/phU_HSgate1
- R61 pad 1: /Project Architecture/Phase W/PhaseW_out -> /Project Architecture/Phase W/phW_HSgate2
- R63 pad 1: /Project Architecture/Phase W/PhaseW_out -> /Project Architecture/Phase W/phW_HSgate2
Routing:
- net /Project Architecture/Phase W/phW_HS: track 0.00 -> 67.4 mm
- net /Project Architecture/Phase U/phU_HS: track 0.00 -> 54.2 mm
- net /Project Architecture/Phase V/phV_HS: track 22.5 -> 67.4 mm
- net /Project Architecture/Phase U/phU_Shunt+: track 0.00 -> 29.5 mm
- net /Project Architecture/Phase W/phW_Shunt+: track 0.00 -> 29.1 mm
- net /Project Architecture/Phase U/phU_Shunt-: track 0.00 -> 28.7 mm
- net /Project Architecture/Phase W/phW_Shunt-: track 0.00 -> 28.2 mm
- net +3.3VA: track 7.31 -> 27.5 mm
- net GND: track 1.05 -> 20.8 mm, vias 60 -> 12
- net Net-(D13-A): track 0.00 -> 15.2 mm
- net Net-(D4-A): track 0.00 -> 15.2 mm
- net Net-(D5-A): track 0.00 -> 15.1 mm
- net Net-(D12-A): track 0.00 -> 15.1 mm
- net Net-(D9-A): track 0.00 -> 15.1 mm
- net /Project Architecture/Phase U/PhaseU_out: track 0.00 -> 10.3 mm
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- added copper zone on B.Cu, net +VSYS
- added copper zone on F.Cu, net +VSYS
- added copper zone on B.Cu, net /Project Architecture/Phase W/phW_HS
- added copper zone on F.Cu, net Net-(R22-Pad2)
- added copper zone on F.Cu, net Net-(R70-Pad2)
- removed copper zone on F.Cu, net (none)
- removed copper zone on F.Cu, net GND
Other:
- board size 190 x 100 mm -> 200 x 100 mm

Commit message: Changing PC
Parts:
- removed the REF** at (64.9, 51.6)
- removed the REF** at (65.0, 64.8)
- removed the REF** at (251.9, 51.6)
- removed the REF** at (252.0, 103.8)
- removed the REF** at (77.9, 51.6)
- removed the REF** at (65.0, 104.0)
- removed the REF** at (251.9, 64.6)
- removed the REF** at (252.0, 130.0)
- removed the REF** at (252.0, 116.9)
- removed the REF** at (65.0, 130.1)
- removed the REF** at (252.0, 90.7)
- removed the REF** at (65.0, 77.9)
- removed the REF** at (78.6, 134.1)
- removed the REF** at (252.0, 77.7)
- removed the REF** at (65.0, 117.0)
- removed the REF** at (65.0, 90.9)
- added H1: MountingHole, MountingHole:MountingHole_4.3mm_M4_Pad_Via, F.Cu at (60.8, 47.4)
- added H2: MountingHole, MountingHole:MountingHole_4.3mm_M4_Pad_Via, F.Cu at (60.7, 137.3)
- added H3: MountingHole, MountingHole:MountingHole_4.3mm_M4_Pad_Via, F.Cu at (250.6, 47.4)
- added H4: MountingHole, MountingHole:MountingHole_4.3mm_M4_Pad_Via, F.Cu at (250.6, 137.2)
- added H5: MountingHole, MountingHole:MountingHole_4.3mm_M4_Pad_Via, F.Cu at (155.7, 47.4)
- added H6: MountingHole, MountingHole:MountingHole_4.3mm_M4_Pad_Via, F.Cu at (155.6, 137.1)
- added H7: MountingHole, MountingHole:MountingHole_4.3mm_M4_Pad_Via, F.Cu at (131.9, 91.8)
- added H8: MountingHole, MountingHole:MountingHole_4.3mm_M4_Pad_Via, F.Cu at (189.5, 91.8)
- added J26: Screw_Terminal_01x01, Bvrny's_library:M8_NutTerminal, F.Cu at (195.6, 45.5)
- added J27: Screw_Terminal_01x01, Bvrny's_library:M8_NutTerminal, F.Cu at (82.3, 122.0)
- added NT1: NetTie_2, NetTie:NetTie-2_SMD_Pad0.5mm, F.Cu at (99.8, 91.8)
- added NT2: NetTie_2, NetTie:NetTie-2_SMD_Pad0.5mm, F.Cu at (105.1, 91.8)
- added NT3: NetTie_2, NetTie:NetTie-2_SMD_Pad0.5mm, F.Cu at (157.5, 91.8)
- added NT4: NetTie_2, NetTie:NetTie-2_SMD_Pad0.5mm, F.Cu at (162.7, 91.8)
- added NT5: NetTie_2, NetTie:NetTie-2_SMD_Pad0.5mm, F.Cu at (214.9, 91.9)
- added NT6: NetTie_2, NetTie:NetTie-2_SMD_Pad0.5mm, F.Cu at (220.2, 91.9)
- added REF**: CP_Radial_D12.5mm_P5.00mm, Capacitor_THT:CP_Radial_D12.5mm_P5.00mm, F.Cu at (59.2, 125.2)
- added REF**: CP_Radial_D12.5mm_P5.00mm, Capacitor_THT:CP_Radial_D12.5mm_P5.00mm, F.Cu at (59.3, 59.0)
- added REF**: CP_Radial_D12.5mm_P5.00mm, Capacitor_THT:CP_Radial_D12.5mm_P5.00mm, F.Cu at (222.6, 135.7)
- added REF**: CP_Radial_D12.5mm_P5.00mm, Capacitor_THT:CP_Radial_D12.5mm_P5.00mm, F.Cu at (246.9, 85.9)
- added REF**: CP_Radial_D12.5mm_P5.00mm, Capacitor_THT:CP_Radial_D12.5mm_P5.00mm, F.Cu at (246.8, 112.2)
- added REF**: CP_Radial_D12.5mm_P5.00mm, Capacitor_THT:CP_Radial_D12.5mm_P5.00mm, F.Cu at (236.2, 50.2)
- added REF**: CP_Radial_D12.5mm_P5.00mm, Capacitor_THT:CP_Radial_D12.5mm_P5.00mm, F.Cu at (59.1, 111.8)
- added REF**: CP_Radial_D12.5mm_P5.00mm, Capacitor_THT:CP_Radial_D12.5mm_P5.00mm, F.Cu at (59.3, 72.2)
- added REF**: CP_Radial_D12.5mm_P5.00mm, Capacitor_THT:CP_Radial_D12.5mm_P5.00mm, F.Cu at (246.9, 72.6)
- added REF**: CP_Radial_D12.5mm_P5.00mm, Capacitor_THT:CP_Radial_D12.5mm_P5.00mm, F.Cu at (59.2, 98.6)
- added REF**: CP_Radial_D12.5mm_P5.00mm, Capacitor_THT:CP_Radial_D12.5mm_P5.00mm, F.Cu at (246.9, 59.4)
- added REF**: CP_Radial_D12.5mm_P5.00mm, Capacitor_THT:CP_Radial_D12.5mm_P5.00mm, F.Cu at (59.2, 85.5)
- added REF**: CP_Radial_D12.5mm_P5.00mm, Capacitor_THT:CP_Radial_D12.5mm_P5.00mm, F.Cu at (246.9, 99.0)
- added REF**: CP_Radial_D12.5mm_P5.00mm, Capacitor_THT:CP_Radial_D12.5mm_P5.00mm, F.Cu at (69.6, 50.1)
- added REF**: CP_Radial_D12.5mm_P5.00mm, Capacitor_THT:CP_Radial_D12.5mm_P5.00mm, F.Cu at (69.7, 135.2)
- added REF**: CP_Radial_D12.5mm_P5.00mm, Capacitor_THT:CP_Radial_D12.5mm_P5.00mm, F.Cu at (222.9, 50.2)
- added REF**: CP_Radial_D12.5mm_P5.00mm, Capacitor_THT:CP_Radial_D12.5mm_P5.00mm, F.Cu at (246.9, 125.5)
- added REF**: CP_Radial_D12.5mm_P5.00mm, Capacitor_THT:CP_Radial_D12.5mm_P5.00mm, F.Cu at (235.9, 135.7)
- moved C154 361.4 mm to (-13.2, 148.9)
- moved C146 221.4 mm to (-16.4, 1.36)
- moved C151 219.6 mm to (-8.90, 175.7)
- moved C152 209.8 mm to (-19.1, 21.2)
- moved C130 144.1 mm to (25.1, 26.9)
- moved C134 144.1 mm to (15.1, 26.7)
- moved C136 144.1 mm to (18.4, 26.8)
- moved C138 144.1 mm to (21.8, 26.9)
- moved C139 144.1 mm to (27.9, 17.5)
- moved C78 144.1 mm to (27.9, 13.5)
- moved C79 144.1 mm to (27.9, 15.5)
- moved C80 144.1 mm to (26.5, 6.06)
- moved C82 144.1 mm to (26.5, 8.08)
- moved C132 144.1 mm to (28.3, 26.9)
- moved C150 138.7 mm to (2.90, 58.2)
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Connections:
- R20 pad 1: /Project Architecture/Phase U/phU_HS -> /Project Architecture/Phase U/PhaseU_out
- R20 pad 2: /Project Architecture/Phase U/phU_Shunt+ -> /Project Architecture/Phase U/phU_HS
- R44 pad 1: /Project Architecture/Phase V/phV_HS -> /Project Architecture/Phase V/PhaseV_out
- R44 pad 2: /Project Architecture/Phase V/phV_Shunt+ -> /Project Architecture/Phase V/phV_HS
- R68 pad 1: /Project Architecture/Phase W/phW_HS -> /Project Architecture/Phase W/PhaseW_out
- R68 pad 2: /Project Architecture/Phase W/phW_Shunt+ -> /Project Architecture/Phase W/phW_HS
Routing:
- net /Project Architecture/Phase W/phW_NTCctrl: track 0.00 -> 15.4 mm
- net GND: track 20.8 -> 17.1 mm
- net /Project Architecture/Phase V/phV_Shunt-: track 28.6 -> 25.4 mm
- net /Project Architecture/Phase V/phV_Shunt+: track 29.4 -> 26.2 mm
- net /Project Architecture/Phase U/phU_Shunt-: track 28.7 -> 25.6 mm
- net /Project Architecture/Phase U/phU_Shunt+: track 29.5 -> 26.5 mm
- net /Project Architecture/Phase W/phW_Shunt-: track 28.2 -> 25.2 mm
- net /Project Architecture/Phase W/phW_Shunt+: track 29.1 -> 26.1 mm
- net Net-(Q20-B): track 0.00 -> 2.74 mm
- net /Project Architecture/Phase V/phV_HS: track 67.4 -> 68.5 mm
- net /Project Architecture/Phase W/phW_HS: track 67.4 -> 68.3 mm
- net /Project Architecture/Phase V/PhaseV_out: vias 0 -> 67
- net /Project Architecture/Phase U/PhaseU_out: vias 0 -> 66
- added copper zone on F.Cu, net GND
