File: PCBA-FLUX-01A/ProjectArchitecture.kicad_sch (KiCad schematic)
At the start: 19 parts, among them J10 Screw_Terminal_01x01, J4 Screw_Terminal_01x01, J5 Screw_Terminal_01x01, J6 Screw_Terminal_01x01, J7 Conn_02x02_Odd_Even, J8 Conn_02x02_Odd_Even, J9 Screw_Terminal_01x01

Commit message: :|
Parts:
- added J1: Conn_02x05_Odd_Even, symbol Connector_Generic:Conn_02x05_Odd_Even
Changed lines of the file:
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@@
 	(text "Inverter"
 		(exclude_from_sim no)
-		(at 214.122 61.722 0)
+		(at 225.298 33.782 0)
 		(effects
 			(font
@@
 	)
 	(symbol
+		(lib_id "Connector_Generic:Conn_02x05_Odd_Even")
+		(at 222.25 106.68 90)
+		(unit 1)
+		(body_style 1)
+		(exclude_from_sim no)
+		(in_bom yes)
+		(on_board yes)
+		(in_pos_files yes)
+		(dnp no)
+		(fields_autoplaced yes)
+		(property "Reference" "J1"
+			(at 229.87 105.4099 90)
+			(show_name no)
+			(do_not_autoplace no)
+			(effects
+				(font
+					(size 1.27 1.27)
+				)
+				(justify right)
+			)
+		)
+		(property "Value" "Conn_02x05_Odd_Even"
+			(at 229.87 106.6799 90)
+			(hide yes)
+			(show_name no)
+			(do_not_autoplace no)
+			(effects
+				(font
+					(size 1.27 1.27)
+				)
+				(justify right)
+			)
+		)
+		(property "Footprint" ""
+			(at 222.25 106.68 0)
+			(hide yes)
+			(show_name no)
+			(do_not_autoplace no)
+			(effects
+				(font
+					(size 1.27 1.27)
+				)
+			)
+		)
+		(property "Datasheet" ""
+			(at 222.25 106.68 0)
+			(hide yes)
+			(show_name no)
+			(do_not_autoplace no)
+			(effects
+				(font
+					(size 1.27 1.27)
+				)
+			)
+		)
+		(property "Description" "Generic connector, double row, 02x05, odd/even pin numbering scheme (row 1 odd numbers, row 2 even numbers), script generated (kicad-library-utils/schlib/autogen/connector/)"
+			(at 222.25 106.68 0)
+			(hide yes)
+			(show_name no)
+			(do_not_autoplace no)
+			(effects
+				(font
+					(size 1.27 1.27)
+				)
+			)
+		)
+		(pin "2"
+		)
+		(pin "8"
+		)
+		(pin "10"
+		)
+		(pin "1"
+		)
+		(pin "3"
+		)
+		(pin "4"
+		)
+		(pin "5"
+		)
+		(pin "6"
+		)
+		(pin "7"
+		)
+		(pin "9"
+		)
+		(instances
+			(project "PCBA-FLUX-01A"
+				(path "/27d049f2-0962-4d9e-88e1-d5cca5250f12/8be822f4-70dc-41bd-a457-afdb13f44dff"
+					(reference "J1")
+					(unit 1)
+				)
+			)
+		)
+	)
+	(symbol
 		(lib_id "Device:C_Polarized")
 		(at 21.59 38.1 0)
@@
 		)
 		(pin "phV_HSgate1" passive
-			(at 241.3 129.54 180)
+			(at 241.3 116.84 180)
 			(effects
 				(font
@@
 		)
 		(pin "phV_HSgate2" passive
-			(at 241.3 134.62 180)
+			(at 241.3 119.38 180)
 			(effects
 				(font
@@
 		)
 		(pin "phV_LSgate1" passive
-			(at 241.3 148.59 180)
+			(at 241.3 124.46 180)
 			(effects
 				(font
@@
 		)
 		(pin "phV_LSgate2" passive
-			(at 241.3 132.08 180)
+			(at 241.3 127 180)
 			(effects
 				(font
@@
 		)
 		(pin "phV_NTCctrl" input
-			(at 241.3 125.73 180)
+			(at 279.4 139.7 0)
 			(effects
 				(font
 					(size 1.27 1.27)
 				)
-				(justify left)
+				(justify right)
 			)
 		)
 		(pin "phV_NTCout" output
-			(at 241.3 118.11 180)
+			(at 241.3 138.43 180)
 			(effects
 				(font
@@
 		)
 		(pin "phV_Voltage" output
-			(at 241.3 127 180)
+			(at 279.4 143.51 0)
 			(effects
 				(font
 					(size 1.27 1.27)
 				)
-				(justify left)
+				(justify right)
 			)
 		)

Commit message: :}
Parts:
- removed J1: Conn_02x05_Odd_Even, symbol Connector_Generic:Conn_02x05_Odd_Even
- added J1, J2: Conn_02x07_Odd_Even, Connector_PinHeader_2.54mm:PinHeader_2x07_P2.54mm_Vertical, symbol Connector_Generic:Conn_02x07_Odd_Even
- added J11: Conn_02x02_Odd_Even, Connector_PinHeader_2.54mm:PinHeader_2x02_P2.54mm_Vertical, symbol Connector_Generic:Conn_02x02_Odd_Even
- added J3: Conn_02x06_Odd_Even, Connector_PinHeader_2.54mm:PinHeader_2x06_P2.54mm_Vertical, symbol Connector_Generic:Conn_02x06_Odd_Even
Connections:
- net GND: now also J1.1 (Pin_1), J1.12 (Pin_12), J1.13 (Pin_13), J1.4 (Pin_4), J1.5 (Pin_5), J1.8 (Pin_8), J1.9 (Pin_9), J11.1 (Pin_1), J11.4 (Pin_4), J2.1 (Pin_1), J2.12 (Pin_12), J2.13 (Pin_13), J2.4 (Pin_4), J2.5 (Pin_5), J2.8 (Pin_8), J2.9 (Pin_9), J3.1 (Pin_1), J3.11 (Pin_11), J3.12 (Pin_12), J3.4 (Pin_4), J3.5 (Pin_5), J3.8 (Pin_8), J3.9 (Pin_9)
- net Phase U/phU_HS: now also J11.3 (Pin_3), J2.3 (Pin_3)
- net Phase U/phU_I+: now also J2.6 (Pin_6)
- net Phase U/phU_I-: now also J2.10 (Pin_10)
- net Phase U/phU_LSgate1: now also J11.2 (Pin_2)
- net Phase U/phU_LSgate2: now also J2.2 (Pin_2)
- net Phase U/phU_Voltage: now also J2.7 (Pin_7)
- net Phase V/PhaseV_out: no longer J5.1 (Pin_1)
- net Phase V/phV_HS: now also J1.3 (Pin_3), J2.11 (Pin_11)
- net Phase V/phV_I+: now also J1.6 (Pin_6)
- net Phase V/phV_I-: now also J1.10 (Pin_10)
- net Phase V/phV_LSgate1: now also J2.14 (Pin_14)
- net Phase V/phV_LSgate2: now also J1.2 (Pin_2)
- net Phase V/phV_Voltage: now also J1.7 (Pin_7)
- net Phase W/PhaseW_out: no longer J6.1 (Pin_1)
- net Phase W/phW_HS: now also J1.11 (Pin_11), J3.3 (Pin_3)
- net Phase W/phW_I+: now also J3.6 (Pin_6)
- net Phase W/phW_I-: now also J3.10 (Pin_10)
- net Phase W/phW_LSgate1: now also J1.14 (Pin_14)
- net Phase W/phW_LSgate2: now also J3.2 (Pin_2)
- net Phase W/phW_Voltage: now also J3.7 (Pin_7)

Commit message: :{
Parts:
- removed J1, J2: Conn_02x07_Odd_Even, Connector_PinHeader_2.54mm:PinHeader_2x07_P2.54mm_Vertical, symbol Connector_Generic:Conn_02x07_Odd_Even
- removed J11: Conn_02x02_Odd_Even, Connector_PinHeader_2.54mm:PinHeader_2x02_P2.54mm_Vertical, symbol Connector_Generic:Conn_02x02_Odd_Even
- removed J3: Conn_02x06_Odd_Even, Connector_PinHeader_2.54mm:PinHeader_2x06_P2.54mm_Vertical, symbol Connector_Generic:Conn_02x06_Odd_Even
- added J1, J11, J12, J13, J14, J15, J16, J17, J18, J19, J2, J3: Conn_01x03_Pin, Connector_PinHeader_2.54mm:PinHeader_1x03_P2.54mm_Vertical, symbol Connector:Conn_01x03_Pin
- added J20, J22, J24: Conn_01x05_Pin, Connector_PinHeader_2.54mm:PinHeader_1x05_P2.54mm_Vertical, symbol Connector:Conn_01x05_Pin
- added J21, J23, J25: Conn_01x04_Pin, Connector_PinHeader_2.54mm:PinHeader_1x04_P2.54mm_Vertical, symbol Connector:Conn_01x04_Pin
Connections:
- net GND: now also J1.2 (Pin_2), J11.2 (Pin_2), J12.2 (Pin_2), J13.2 (Pin_2), J14.2 (Pin_2), J15.2 (Pin_2), J16.2 (Pin_2), J17.2 (Pin_2), J18.2 (Pin_2), J19.2 (Pin_2), J2.2 (Pin_2), J20.2 (Pin_2), J20.4 (Pin_4), J21.4 (Pin_4), J22.2 (Pin_2), J22.4 (Pin_4), J23.4 (Pin_4), J24.2 (Pin_2), J24.4 (Pin_4), J25.4 (Pin_4), J3.2 (Pin_2)
- net Phase U/PhaseU_out: now also J4.1 (Pin_1)
- net Phase U/phU_HS: now also J1.3 (Pin_3), J11.1 (Pin_1), J2.3 (Pin_3), J3.1 (Pin_1)
- net Phase U/phU_I+: now also J24.3 (Pin_3)
- net Phase U/phU_I-: now also J24.1 (Pin_1)
- net Phase U/phU_LSgate1: now also J3.3 (Pin_3)
- net Phase U/phU_LSgate2: now also J11.3 (Pin_3)
- net Phase U/phU_Voltage: now also J24.5 (Pin_5)
- net Phase V/PhaseV_out: now also J5.1 (Pin_1)
- net Phase V/phV_HS: now also J12.3 (Pin_3), J13.3 (Pin_3), J14.1 (Pin_1), J15.1 (Pin_1)
- net Phase V/phV_HSgate1: now also J12.1 (Pin_1)
- net Phase V/phV_HSgate2: now also J13.1 (Pin_1)
- net Phase V/phV_I+: now also J22.3 (Pin_3)
- net Phase V/phV_I-: now also J22.1 (Pin_1)
- net Phase V/phV_LSgate1: now also J14.3 (Pin_3)
- net Phase V/phV_LSgate2: now also J15.3 (Pin_3)
- net Phase V/phV_NTCctrl: now also J23.3 (Pin_3)
- net Phase V/phV_NTCout: now also J23.2 (Pin_2)
- net Phase V/phV_Voltage: now also J22.5 (Pin_5)
- net Phase W/PhaseW_out: now also J6.1 (Pin_1)
- net Phase W/phW_HS: now also J16.3 (Pin_3), J17.3 (Pin_3), J18.1 (Pin_1), J19.1 (Pin_1)
- net Phase W/phW_HSgate1: now also J16.1 (Pin_1)
- net Phase W/phW_I+: now also J20.3 (Pin_3)
- net Phase W/phW_I-: now also J20.1 (Pin_1)
- net Phase W/phW_LSgate1: now also J18.3 (Pin_3)
- net Phase W/phW_LSgate2: now also J19.3 (Pin_3)
- net Phase W/phW_NTCctrl: now also J21.2 (Pin_2)
- net Phase W/phW_NTCout: now also J21.3 (Pin_3)
- net Phase W/phW_Voltage: now also J20.5 (Pin_5)
- new net +3.3VA: J21.1 (Pin_1), J23.1 (Pin_1), J25.1 (Pin_1)
- new net Phase U/phU_HSgate1: J1.1 (Pin_1)
- new net Phase U/phU_HSgate2: J2.1 (Pin_1)
- new net Phase U/phU_NTCctrl: J25.2 (Pin_2)
- new net Phase U/phU_NTCout: J25.3 (Pin_3)
- new net Phase W/phW_HSgate2: J17.1 (Pin_1)
Other:
- moved on the sheet: C143, C144, C145, C146, C147, C148, C149, C150, C151, C152, C153, C154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
