File: PCBA-FLUX-01A/PhaseU.kicad_sch (KiCad schematic)
At the start: 47 parts, among them Q18 BC860C, Q2 IPT015N10N5, Q3 IPT015N10N5, Q4 IPT015N10N5, Q5 IPT015N10N5

Commit message: :{
Parts:
- removed C112, C113, C114, C115, C116: 10uF, Capacitor_SMD:C_1210_3225Metric, symbol Device:C
- removed C117, C43, C45, C47, C50: 100nF, Capacitor_SMD:C_0805_2012Metric, symbol Device:C
- removed NT1: NetTie_2, NetTie:NetTie-2_SMD_Pad0.5mm, symbol Device:NetTie_2
- added C56: 3.3nF, Capacitor_SMD:C_0603_1608Metric, symbol Device:C
- added R26, R27: 51k, Resistor_SMD:R_0805_2012Metric, symbol Device:R
- added R34: 4k7, Resistor_SMD:R_0805_2012Metric, symbol Device:R
Connections:
- net GND: now also C56.2, R34.2
- net PhaseU_out: now also R26.1
- net phU_Voltage: now also C56.1, R27.2, R34.1
- new net: R26.2, R27.1
Other:
- note removed: "DC-Link"

Commit message: Changing PC
Parts:
- removed R20: 0.1mR, Bvrny's_library:R5930, symbol Device:R_Shunt
- added NT1, NT2: NetTie_2, NetTie:NetTie-2_SMD_Pad0.5mm, symbol Device:NetTie_2
- added R20: 0.1mR, Bvrny's_library:R5930, symbol Device:R
Connections:
- net PhaseU_out: now also NT2.2, R20.1
- net phU_HS: now also NT1.2, R20.2
- net phU_Shunt+: now also NT1.1
- net phU_Shunt-: now also NT2.1
