File: PCBA-FLUX-01A/PhaseV.kicad_sch (KiCad schematic)
At the start: 50 parts, among them Q19 BC860C, Q6 IPT015N10N5, Q7 IPT015N10N5, Q8 IPT015N10N5, Q9 IPT015N10N5

Commit message: :{
Parts:
- removed C119, C121, C123, C125, C127, C140, C141: 10uF, Capacitor_SMD:C_1210_3225Metric, symbol Device:C
- removed C128, C142, C60, C61, C62, C64: 100nF, Capacitor_SMD:C_0805_2012Metric, symbol Device:C
- removed NT2: NetTie_2, NetTie:NetTie-2_SMD_Pad0.5mm, symbol Device:NetTie_2
- added C57: 3.3nF, Capacitor_SMD:C_0603_1608Metric, symbol Device:C
- added R35, R36: 51k, Resistor_SMD:R_0805_2012Metric, symbol Device:R
- added R43: 4k7, Resistor_SMD:R_0805_2012Metric, symbol Device:R
Connections:
- net GND: now also C57.2, R43.2
- net PhaseV_out: now also R35.1
- net phV_Voltage: now also C57.1, R36.2, R43.1
- new net: R35.2, R36.1
Other:
- note removed: "DC-Link"

Commit message: Changing PC
Parts:
- removed R44: 0.1mR, Bvrny's_library:R5930, symbol Device:R_Shunt
- added NT3, NT4: NetTie_2, NetTie:NetTie-2_SMD_Pad0.5mm, symbol Device:NetTie_2
- added R44: 0.1mR, Bvrny's_library:R5930, symbol Device:R
Connections:
- net PhaseV_out: now also NT4.2, R44.1
- net phV_HS: now also NT3.2, R44.2
- net phV_Shunt+: now also NT3.1
- net phV_Shunt-: now also NT4.1
