File: PCBA-FLUX-01A/PhaseW.kicad_sch (KiCad schematic)
At the start: 47 parts, among them Q10 IPT015N10N5, Q11 IPT015N10N5, Q12 IPT015N10N5, Q13 IPT015N10N5, Q20 BC860C

Commit message: :{
Parts:
- removed NT3: NetTie_2, NetTie:NetTie-2_SMD_Pad0.5mm, symbol Device:NetTie_2
- added C58: 3.3nF, Capacitor_SMD:C_0603_1608Metric, symbol Device:C
- added R49, R50: 51k, Resistor_SMD:R_0805_2012Metric, symbol Device:R
- added R51: 4k7, Resistor_SMD:R_0805_2012Metric, symbol Device:R
Connections:
- net GND: now also C58.2, R51.2
- net PhaseW_out: now also R49.1
- net phW_Voltage: now also C58.1, R50.2, R51.1
- new net: R49.2, R50.1

Commit message: Changing PC
Parts:
- removed R68: 0.1mR, Bvrny's_library:R5930, symbol Device:R_Shunt
- added NT5, NT6: NetTie_2, NetTie:NetTie-2_SMD_Pad0.5mm, symbol Device:NetTie_2
- added R68: 0.1mR, Bvrny's_library:R5930, symbol Device:R
Connections:
- net PhaseW_out: now also NT6.2, R68.1
- net phW_HS: now also NT5.2, R68.2
- net phW_Shunt+: now also NT5.1
- net phW_Shunt-: now also NT6.1
