File: PCBA-VECTOR-01A/PCBA-VECTOR-01A.kicad_sch (KiCad schematic)
At the start: 0 parts

Commit message: Finished inverter design and started working on MCU pin out
Other:
- added sheet Block Diagram (BlockDiagram.kicad_sch)
- added sheet Project Architecture (ProjectArchitecture.kicad_sch)
- added sheet Revision History (RevisionHistory.kicad_sch)
- note added: "..............."
- note added: "1"
- note added: "10"
- note added: "11"
- note added: "12"
- note added: "13"
- note added: "14"
- note added: "15"
- note added: "16"
- note added: "17"
- note added: "18"
- note added: "19"
- note added: "2"
- note added: "20"
- note added: "2026-05-26"
- note added: "21"
- note added: "22"
- note added: "23"
- note added: "24"
- note added: "25"
- note added: "26"
- note added: "27"
- note added: "28"
- note added: "29"
- note added: "3"
- note added: "30"
- note added: "31"
- note added: "32"
- note added: "33"
- note added: "34"
- note added: "35"
- note added: "36"
- note added: "37"
- note added: "38"
- note added: "39"
- note added: "4"
- note added: "40"
- note added: "5"
- note added: "6"
- note added: "7"
- note added: "8"
- note added: "9"
- note added: "BOTTOM VIEW"
- note added: "Block Diagram"
- note added: "CHECKED - There shouldn't be any mistakes. Contact the engineer if you find any."
- note added: "Comment"
- note added: "Cover Page"
- note added: "DESIGN CONSIDERATIONS"
- note added: "DRAFT - Very early stage of schematic, ignore details."
- note added: "Index"
- note added: "NAME"
- note added: "NOTES"
- note added: "Not fitted components are marked as"
- note added: "PRELIMINARY - Close to final schematic."
- note added: "Page"
- note added: "Project Architecture"
- note added: "RELEASED - A board with this schematic has been sent to production."
- note added: "Rev 1.0.0"
- note added: "Revison History"
- note added: "TOP VIEW"
- note added: "Variant: DRAFT"
