File: PCBA-VECTOR-01A/PCBA-VECTOR-01A.kicad_sch (KiCad schematic)
At the start: 0 parts

Commit message: Changes were made
Other:
- note added: "2026-07-06"
- note added: "Comm's"
- note added: "MCU"
- note added: "Motor Output"
- note added: "Power Input"
- note added: "Power Supply"
- note added: "Vector"
- note removed: "2026-05-26"
- note removed: "NAME"
- company: (none) -> Jovanovski Laboratory - JLab
