File: PCBA-VECTOR-01A/RevisionHistory.kicad_sch (KiCad schematic)
At the start: 0 parts

Commit message: Changes were made
Other:
- company: (none) -> Jovanovski Laboratory - JLab
Changed lines of the file:
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@@
 	(generator_version "10.0")
 	(paper "A4")
+	(title_block
+		(rev "1.0.0")
+		(company "Jovanovski Laboratory - JLab")
+		(comment 1 "Bvrny")
+		(comment 3 "Vector")
+		(comment 4 "Vortex")
+	)
 )
