File: PCBA-VECTOR-01A/Comms.kicad_sch (KiCad schematic)
At the start: 26 parts, among them J16 Conn_01x02_Pin, J18 Screw_Terminal_01x03, J20 Conn_01x02_Pin, J21 Screw_Terminal_01x03, U12 MCP2551-I-SN, U14 ST485EDR, U17 TYPE-C 16PLT-H10.0, U9 NUP4114

Commit message: Changes were made
Parts:
- added C116, C117: 100nF, Capacitor_SMD:C_0402_1005Metric, symbol Device:C
- added J1: Screw_Terminal_01x06, Bvrny's_library:TerminalBlock_5.08_01x06_JLAB, symbol Connector:Screw_Terminal_01x06
- added J6: Conn_01x03_Pin, Connector_PinHeader_2.54mm:PinHeader_1x03_P2.54mm_Vertical, symbol Connector:Conn_01x03_Pin
- added J8: Screw_Terminal_01x04, Bvrny's_library:TerminalBlock_5.08_01x04_JLAB, symbol Connector:Screw_Terminal_01x04
- added U10, U11: NUP4114, Package_SO:TSOP-6_1.65x3.05mm_P0.95mm, symbol Bvrny's_library:NUP4114
Connections:
- net +3.3V: now also C116.1, C117.1, J1.1 (Pin_1), J8.1 (Pin_1), U10.5 (VCC), U11.5 (VCC)
- net GND: now also C116.2, C117.2, J1.6 (Pin_6), J6.3 (Pin_3), J8.4 (Pin_4), U10.2 (GND), U11.2 (GND)
- net USB_D+ renamed D+
- net USB_D- renamed D-
- new net SCL: J8.2 (Pin_2), U11.4 (I/O4)
- new net SDA: J8.3 (Pin_3), U11.3 (I/O3)
- new net SPI1_MISO: J1.4 (Pin_4), U10.6 (I/O2)
- new net SPI1_MOSI: J1.3 (Pin_3), U10.4 (I/O4)
- new net SPI1_NSS: J1.5 (Pin_5), U10.1 (I/O1)
- new net SPI1_SCK: J1.2 (Pin_2), U10.3 (I/O3)
- new net USART1_RXD: J6.2 (Pin_2), U11.1 (I/O1)
- new net USART1_TXD: J6.1 (Pin_1), U11.6 (I/O2)
Other:
- company: (none) -> Jovanovski Laboratory - JLab
- moved on the sheet: C48, C49, R31, R32, U17, U9

Commit message: Finished schematic?
Parts:
- removed J6: Conn_01x03_Pin, Connector_PinHeader_2.54mm:PinHeader_1x03_P2.54mm_Vertical, symbol Connector:Conn_01x03_Pin
- added C118: 100nF, Capacitor_SMD:C_0402_1005Metric, symbol Device:C
- added J13: Screw_Terminal_01x04, Bvrny's_library:TerminalBlock_5.08_01x04_JLAB, symbol Connector:Screw_Terminal_01x04
Connections:
- net +3.3V: now also C118.1, J13.1 (Pin_1)
- net GND: now also C118.2, J13.4 (Pin_4)
- net USART1_RXD: now also J13.3 (Pin_3)
- net USART1_TXD: now also J13.2 (Pin_2)
Other:
- note added: "CAN Bus"
- note added: "RS485/Modbus RTU"
- note added: "SPI"
- note added: "UART & I2C"
- note added: "USB2.0 Type-C"
- note removed: "CAN bus communication"
- note removed: "Modbus RTU - RS485 communication"
- moved on the sheet: C114, C115, C116, C117, C48, C49, C88, C90, C93, C95, C96, D7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
