File: PCBA-VECTOR-01A/PowerInput.kicad_sch (KiCad schematic)
At the start: 3 parts, among them J10 Conn_02x06_Odd_Even, J11 Conn_02x06_Odd_Even, J9 Conn_02x06_Odd_Even

Commit message: Changes were made
Parts:
- removed J10, J11, J9: Conn_02x06_Odd_Even, Connector_PinHeader_2.54mm:PinHeader_2x06_P2.54mm_Vertical, symbol Connector_Generic:Conn_02x06_Odd_Even
- added D13: SMBJ60A-13-F, Diode_SMD:D_SMB, symbol Synapse:SMBJ60A
- added D14: SK1010C, Diode_SMD:D_SMC, symbol Synapse:D_Schottky
- added D23: Red LED, LED_SMD:LED_0603_1608Metric, symbol Synapse:LED
- added F1: Fuse, Fuse:Fuseholder_Cylinder-5x20mm_Stelvio-Kontek_PTF78_Horizontal_Open, symbol Synapse:Fuse
- added J5, J7: Conn_02x02_Odd_Even, Connector_PinSocket_2.54mm:PinSocket_2x02_P2.54mm_Vertical, symbol Connector_Generic:Conn_02x02_Odd_Even
- added R104: 5.1K, Resistor_SMD:R_0402_1005Metric, symbol Synapse:R
Connections:
- net GND: now also D13.2, J7.1 (Pin_1), J7.2 (Pin_2), J7.3 (Pin_3), J7.4 (Pin_4), R104.2
- new net: D23.1 (K), R104.1
- new net: D14.2 (A), F1.2
- new net +VBATT: F1.1, J5.1 (Pin_1), J5.2 (Pin_2), J5.3 (Pin_3), J5.4 (Pin_4)
- new net +VSYS: D13.1, D14.1 (K), D23.2 (A)
Other:
- removed sheet Comm's
- removed sheet MCU
- removed sheet Motor Output
- removed sheet Power Input
- removed sheet Power Supply

Commit message: Finished schematic?
Parts:
- removed D13: SMBJ60A-13-F, Diode_SMD:D_SMB, symbol Synapse:SMBJ60A
- removed R104: 5.1K, Resistor_SMD:R_0402_1005Metric, symbol Synapse:R
- added C51: 3.3nF, Capacitor_SMD:C_0603_1608Metric, symbol Device:C
- added C52: 100nF, Capacitor_SMD:C_0402_1005Metric, symbol Device:C
- added C53: 1nF, Capacitor_SMD:C_0603_1608Metric, symbol Device:C
- added D2: SMCJ70A, Diode_SMD:D_SMC, symbol Bvrny's_library:SMCJ70A
- added R10, R21: 51k, Resistor_SMD:R_0805_2012Metric, symbol Device:R
- added R22: 4k7, Resistor_SMD:R_0805_2012Metric, symbol Device:R
- added R23: 100R, Resistor_SMD:R_0603_1608Metric, symbol Device:R
- added R9: 25.5K, Resistor_SMD:R_0603_1608Metric, symbol Device:R
- added U7: TLV9001, Package_TO_SOT_SMD:SOT-23-5, symbol Bvrny's_library:TLV9001IDBVR
Connections:
- net +VSYS: now also D2.1, R10.1
- net GND: now also C51.2, C52.2, C53.2, D2.2, R22.2, R9.2, U7.5 (V_{SS})
- net at D23.1 (K): now also R9.1
- new net: C51.1, R21.2, R22.1, U7.3 (IN+)
- new net: R10.2, R21.1
- new net: R23.1, U7.1 (OUT), U7.4 (IN-)
- new net +3.3VA: C52.1, U7.2 (V_{DD})
- new net Vsys: C53.1, R23.2
Other:
- note added: "Battery Voltage"
- note added: "Board connectors for power to Flux"
- note added: "Input protection"
- moved on the sheet: D14, D23, F1, J5, J7
