File: PCBA-VECTOR-01A/AnalogFrontend.kicad_sch (KiCad schematic)
At the start: 4 parts, among them J10 Conn_02x06_Odd_Even, J11 Conn_02x06_Odd_Even, J12 Conn_02x06_Odd_Even, J9 Conn_02x06_Odd_Even

Commit message: Moved the current and voltage sensing OpAmp's to Vector
Parts:
- removed J10, J11, J12, J9: Conn_02x06_Odd_Even, Connector_PinHeader_2.54mm:PinHeader_2x06_P2.54mm_Vertical, symbol Connector_Generic:Conn_02x06_Odd_Even
- added C29, C54, C57, C59, C60, C62, C63, C66, C69: 100nF, Capacitor_SMD:C_0402_1005Metric, symbol Device:C
- added C55, C61, C64: 2.2nF, Capacitor_SMD:C_0603_1608Metric, symbol Device:C
- added C56, C65, C68: 3.3nF, Capacitor_SMD:C_0603_1608Metric, symbol Device:C
- added C58, C67, C70: 1nF, Capacitor_SMD:C_0603_1608Metric, symbol Device:C
- added R24, R29, R30: 100R, palmkiLib:R_0603_1608Metric, symbol Device:R
- added R25, R26, R33, R34, R37, R38: 51k, Resistor_SMD:R_0805_2012Metric, symbol Device:R
- added R27, R35, R39: 4k7, Resistor_SMD:R_0805_2012Metric, symbol Device:R
- added R28, R36, R40: 100R, Resistor_SMD:R_0603_1608Metric, symbol Device:R
- added U15, U19, U20: TLV9001, Package_TO_SOT_SMD:SOT-23-5, symbol Bvrny's_library:TLV9001IDBVR
- added U16, U18, U8: INA240A2DR, Package_SO:SOIC-8_3.9x4.9mm_P1.27mm, symbol Bvrny's_library:INA240A2DR
Connections:
- net GND: now also C29.2, C54.2, C55.2, C56.2, C57.2, C58.2, C59.2, C60.2, C61.2, C62.2, C63.2, C64.2, C65.2, C66.2, C67.2, C68.2, C69.2, C70.2, R27.2, R35.2, R39.2, U15.5 (V_{SS}), U16.2 (GND), U16.4 (NC), U16.7 (REF1), U18.2 (GND), U18.4 (NC), U18.7 (REF1), U19.5 (V_{SS}), U20.5 (V_{SS}), U8.2 (GND), U8.4 (NC), U8.7 (REF1)
- new net: R37.2, R38.1
- new net: C68.1, R38.2, R39.1, U20.3 (IN+)
- new net: R28.1, U15.1 (OUT), U15.4 (IN-)
- new net: C56.1, R26.2, R27.1, U15.3 (IN+)
- new net: R24.1, U8.5 (OUT)
- new net: C65.1, R34.2, R35.1, U19.3 (IN+)
- new net: R36.1, U19.1 (OUT), U19.4 (IN-)
- new net: R29.1, U16.5 (OUT)
- new net: R40.1, U20.1 (OUT), U20.4 (IN-)
- new net: R33.2, R34.1
- new net: R25.2, R26.1
- new net: R30.1, U18.5 (OUT)
- new net +3.3VA: C29.1, C54.1, C57.1, C59.1, C60.1, C62.1, C63.1, C66.1, C69.1, U15.2 (V_{DD}), U16.3 (REF2), U16.6 (VS), U18.3 (REF2), U18.6 (VS), U19.2 (V_{DD}), U20.2 (V_{DD}), U8.3 (REF2), U8.6 (VS)
- new net phU_I+: U8.8 (IN+)
- new net phU_I-: U8.1 (IN-)
- new net phU_V: R25.1
- new net phU_current: C55.1, R24.2
- new net phU_voltage: C58.1, R28.2
- new net phV_I+: U16.8 (IN+)
- new net phV_I-: U16.1 (IN-)
- new net phV_V: R33.1
- new net phV_current: C61.1, R29.2
- new net phV_voltage: C67.1, R36.2
- new net phW_I+: U18.8 (IN+)
- new net phW_I-: U18.1 (IN-)
- new net phW_V: R37.1
- new net phW_current: C64.1, R30.2
- new net phW_voltage: C70.1, R40.2
Other:
- removed sheet Analog Frontend
- removed sheet Comm's
- removed sheet MCU
- removed sheet Motor Output
- removed sheet Power Input
- removed sheet Power Supply
- note added: "Phase U Current Sense"
- note added: "Phase U Voltage"
- note added: "Phase V Current Sense"
- note added: "Phase V Voltage"
- note added: "Phase W Current Sense"
- note added: "Phase W Voltage"
- note removed: "Board connectors to Flux"
- company: Jovanovski Laboratory - JLab -> (none)
