File: PCBA-VECTOR-01A/GateDrivers.kicad_sch (KiCad schematic)
At the start: 19 parts, among them J10 Screw_Terminal_01x01, J4 Screw_Terminal_01x01, J5 Screw_Terminal_01x01, J6 Screw_Terminal_01x01, J7 Conn_02x02_Odd_Even, J8 Conn_02x02_Odd_Even, J9 Screw_Terminal_01x01

Commit message: More routing on FLux
Parts:
- removed C143, C144, C145, C146, C147, C148, C149, C150, C151, C152, C153, C154: 1000uF, Capacitor_THT:CP_Radial_D18.0mm_P7.50mm, symbol Device:C_Polarized
- removed J10, J4, J5, J6, J9: Screw_Terminal_01x01, Bvrny's_library:M8_NutTerminal, symbol Connector:Screw_Terminal_01x01
- removed J7, J8: Conn_02x02_Odd_Even, Connector_PinHeader_2.54mm:PinHeader_2x02_P2.54mm_Vertical, symbol Connector_Generic:Conn_02x02_Odd_Even
- added C100, C106, C107, C113, C122, C99: 1nF, Capacitor_SMD:C_0603_1608Metric, symbol Device:C
- added C101, C103, C108, C110, C123, C125: 100nF, Capacitor_SMD:C_0402_1005Metric, symbol Device:C
- added C102, C109, C124: 2.2uF, Capacitor_SMD:C_1206_3216Metric, symbol Device:C
- added C104, C105, C111, C112, C71, C86: 22uF, Capacitor_SMD:C_1206_3216Metric, symbol Device:C
- added R1, R41, R42, R43, R44, R45: 100R, Resistor_SMD:R_0603_1608Metric, symbol Device:R
- added U21, U22, U23: UCC27211AQDDARQ1, Package_SO:SOIC-8-1EP_3.9x4.9mm_P1.27mm_EP2.95x4.9mm_Mask2.34x2.34mm_ThermalVias, symbol Bvrny's_library:UCC27211AQDDARQ1
Connections:
- net GND: now also C100.2, C101.2, C104.2, C105.2, C106.2, C107.2, C108.2, C111.2, C112.2, C113.2, C122.2, C123.2, C71.2, C86.2, C99.2, U21.7 (VSS), U21.9 (Pad), U22.7 (VSS), U22.9 (Pad), U23.7 (VSS), U23.9 (Pad)
- new net: C99.1, R1.2, U21.5 (HI)
- new net: C106.1, R42.2, U22.5 (HI)
- new net: C107.1, R43.2, U22.6 (LI)
- new net: C113.1, R44.2, U23.5 (HI)
- new net: C122.1, R45.2, U23.6 (LI)
- new net: C100.1, R41.2, U21.6 (LI)
- new net +12V: C101.1, C104.1, C105.1, C108.1, C111.1, C112.1, C123.1, C71.1, C86.1, U21.1 (VDD), U22.1 (VDD), U23.1 (VDD)
- new net phU_HB: C102.1, C103.1, U21.2 (HB)
- new net phU_HI: R1.1
- new net phU_HS: C102.2, C103.2, U21.4 (HS)
- new net phU_HSgate: U21.3 (HO)
- new net phU_LI: R41.1
- new net phU_LSgate: U21.8 (LO)
- new net phV_HB: C109.1, C110.1, U22.2 (HB)
- new net phV_HI: R42.1
- new net phV_HS: C109.2, C110.2, U22.4 (HS)
- new net phV_HSgate: U22.3 (HO)
- new net phV_LI: R43.1
- new net phV_LSgate: U22.8 (LO)
- new net phW_HB: C124.1, C125.1, U23.2 (HB)
- new net phW_HI: R44.1
- new net phW_HS: C124.2, C125.2, U23.4 (HS)
- new net phW_HSgate: U23.3 (HO)
- new net phW_LI: R45.1
- new net phW_LSgate: U23.8 (LO)
Other:
- removed sheet Phase U
- removed sheet Phase V
- removed sheet Phase W
- note added: "Phase U gate driver"
- note added: "Phase V gate driver"
- note added: "Phase W gate driver"
- note removed: "Board connectors for power to Vector"
- note removed: "Board connectors to Vector"
- note removed: "High current connectors"
- note removed: "Inverter"
- note removed: "Power input connectors"
- company: Jovanovski Laboratory - JLAB -> (none)
