File: PCBA-FLUX-01A/_restore_backup_2026-08-06T12-56-59-886/BlockDiagram.kicad_sch (KiCad schematic)
At the start: 19 parts, among them J10 Screw_Terminal_01x01, J4 Screw_Terminal_01x01, J5 Screw_Terminal_01x01, J6 Screw_Terminal_01x01, J7 Conn_02x02_Odd_Even, J8 Conn_02x02_Odd_Even, J9 Screw_Terminal_01x01

Commit message: More routing on FLux
Parts:
- removed C143, C144, C145, C146, C147, C148, C149, C150, C151, C152, C153, C154: 1000uF, Capacitor_THT:CP_Radial_D18.0mm_P7.50mm, symbol Device:C_Polarized
- removed J10, J4, J5, J6, J9: Screw_Terminal_01x01, Bvrny's_library:M8_NutTerminal, symbol Connector:Screw_Terminal_01x01
- removed J7, J8: Conn_02x02_Odd_Even, Connector_PinHeader_2.54mm:PinHeader_2x02_P2.54mm_Vertical, symbol Connector_Generic:Conn_02x02_Odd_Even
Other:
- removed sheet Phase U
- removed sheet Phase V
- removed sheet Phase W
- note removed: "Board connectors for power to Vector"
- note removed: "Board connectors to Vector"
- note removed: "High current connectors"
- note removed: "Inverter"
- note removed: "Power input connectors"
