File: PCBA-FLUX-01A/_restore_backup_2026-08-06T12-56-59-886/PCBA-FLUX-01A.kicad_pcb (KiCad board)
At the start: 2 copper layers, 160 x 100 mm, 164 parts, among them J10 Screw_Terminal_01x01, J4 Screw_Terminal_01x01, J5 Screw_Terminal_01x01, J6 Screw_Terminal_01x01, J7 Conn_02x02_Odd_Even, J8 Conn_02x02_Odd_Even, J9 Screw_Terminal_01x01, Q10 IPT015N10N5, Q11 IPT015N10N5, Q12 IPT015N10N5, Q13 IPT015N10N5, Q18 BC860C, Q19 BC860C, Q2 IPT015N10N5, Q20 BC860C, Q3 IPT015N10N5, Q4 IPT015N10N5, Q5 IPT015N10N5, Q6 IPT015N10N5, Q7 IPT015N10N5, Q8 IPT015N10N5, Q9 IPT015N10N5

Commit message: More routing on FLux
Parts:
- removed the REF** at (114.7, 108.9)
- added REF**: PinHeader_2x05_P2.54mm_Vertical, Connector_PinHeader_2.54mm:PinHeader_2x05_P2.54mm_Vertical, F.Cu at (109.6, 107.4)
- moved J4 4.69 mm to (74.8, 148.2)
- moved C101 3.70 mm to (205.2, 133.7)
- moved J5 3.70 mm to (125.8, 148.4)
- moved J6 3.70 mm to (178.0, 148.3)
- moved NT1 3.70 mm to (96.8, 133.2)
- moved R81 3.70 mm to (148.5, 133.6)
- moved D3 3.70 mm to (66.6, 119.3)
- moved D5 3.70 mm to (111.2, 119.3)
- moved Q3 3.70 mm to (75.4, 115.8)
- moved Q5 3.70 mm to (102.4, 115.9)
- moved Q7 3.70 mm to (127.0, 115.9)
- moved Q9 3.70 mm to (153.9, 115.8)
- moved R14 3.70 mm to (113.5, 113.5)
- moved R16 3.70 mm to (111.2, 113.5)
- moved R19 3.70 mm to (108.9, 113.5)
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Routing:
- net /Project Architecture/Phase W/phW_HS: vias 98 -> 0
- net /Project Architecture/Phase V/phV_Shunt+: vias 1 -> 0
- net /Project Architecture/Phase V/phV_HS: vias 99 -> 0
- net /Project Architecture/Phase U/phU_HS: vias 97 -> 0
- net +VSYS: vias 224 -> 0
- removed copper zone on B.Cu, net +VSYS
