File: PCBA-FLUX-01A/_restore_backup_2026-08-06T12-56-59-886/PCBA-FLUX-01A.kicad_sch (KiCad schematic)
At the start: 19 parts, among them J10 Screw_Terminal_01x01, J4 Screw_Terminal_01x01, J5 Screw_Terminal_01x01, J6 Screw_Terminal_01x01, J7 Conn_02x02_Odd_Even, J8 Conn_02x02_Odd_Even, J9 Screw_Terminal_01x01

Commit message: More routing on FLux
Parts:
- removed C143, C144, C145, C146, C147, C148, C149, C150, C151, C152, C153, C154: 1000uF, Capacitor_THT:CP_Radial_D18.0mm_P7.50mm, symbol Device:C_Polarized
- removed J10, J4, J5, J6, J9: Screw_Terminal_01x01, Bvrny's_library:M8_NutTerminal, symbol Connector:Screw_Terminal_01x01
- removed J7, J8: Conn_02x02_Odd_Even, Connector_PinHeader_2.54mm:PinHeader_2x02_P2.54mm_Vertical, symbol Connector_Generic:Conn_02x02_Odd_Even
Other:
- removed sheet Phase U
- removed sheet Phase V
- removed sheet Phase W
- added sheet Block Diagram (BlockDiagram.kicad_sch)
- added sheet Project Architecture (ProjectArchitecture.kicad_sch)
- added sheet Revision History (RevisionHistory.kicad_sch)
- note added: "..............."
- note added: "1"
- note added: "10"
- note added: "11"
- note added: "12"
- note added: "13"
- note added: "14"
- note added: "15"
- note added: "16"
- note added: "17"
- note added: "18"
- note added: "19"
- note added: "2"
- note added: "20"
- note added: "2026-07-06"
- note added: "21"
- note added: "22"
- note added: "23"
- note added: "24"
- note added: "25"
- note added: "26"
- note added: "27"
- note added: "28"
- note added: "29"
- note added: "3"
- note added: "30"
- note added: "31"
- note added: "32"
- note added: "33"
- note added: "34"
- note added: "35"
- note added: "36"
- note added: "37"
- note added: "38"
- note added: "39"
- note added: "4"
- note added: "40"
- note added: "5"
- note added: "6"
- note added: "7"
- note added: "8"
- note added: "9"
- note added: "BOTTOM VIEW"
- note added: "Block Diagram"
- note added: "CHECKED - There shouldn't be any mistakes. Contact the engineer if you find any."
- note added: "Comment"
- note added: "Cover Page"
- note added: "DESIGN CONSIDERATIONS"
- note added: "DRAFT - Very early stage of schematic, ignore details."
- note added: "FLUX"
- note added: "Index"
- note added: "NOTES"
- note added: "Not fitted components are marked as"
- note added: "PRELIMINARY - Close to final schematic."
- note added: "Page"
- note added: "Phase U"
- note added: "Phase V"
- note added: "Phase W"
- note added: "Project Architecture"
- note added: "RELEASED - A board with this schematic has been sent to production."
- note added: "Rev 1.0.0"
- note added: "Revison History"
- note added: "TOP VIEW"
- note added: "Variant: DRAFT"
- note removed: "Board connectors for power to Vector"
- note removed: "Board connectors to Vector"
- note removed: "High current connectors"
- note removed: "Inverter"
- note removed: "Power input connectors"
