File: PCBA-FLUX-01A/_restore_backup_2026-08-06T12-56-59-886/ProjectArchitecture.kicad_sch (KiCad schematic)
At the start: 19 parts, among them J10 Screw_Terminal_01x01, J4 Screw_Terminal_01x01, J5 Screw_Terminal_01x01, J6 Screw_Terminal_01x01, J7 Conn_02x02_Odd_Even, J8 Conn_02x02_Odd_Even, J9 Screw_Terminal_01x01

Commit message: More routing on FLux
Other:
- sheet Phase U ports: added none; removed phU_Voltage
- sheet Phase V ports: added none; removed phV_HS, phV_HSgate1, phV_HSgate2, phV_I+, phV_I-, phV_LSgate1, phV_LSgate2, phV_NTCctrl, phV_NTCout, phV_Voltage
- sheet Phase W ports: added none; removed phW_HS, phW_HSgate1, phW_HSgate2, phW_I+, phW_I-, phW_LSgate1, phW_LSgate2, phW_NTCctrl, phW_NTCout, phW_Voltage
- moved on the sheet: J6
Changed lines of the file:
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@@
 	(wire
 		(pts
-			(xy 279.4 129.54) (xy 344.17 129.54)
+			(xy 270.51 129.54) (xy 344.17 129.54)
 		)
 		(stroke
@@
 	(wire
 		(pts
-			(xy 279.4 176.53) (xy 345.44 176.53)
+			(xy 270.51 167.64) (xy 344.17 167.64)
 		)
 		(stroke
@@
 	)
 	(image
-		(at 359.41 176.53)
+		(at 358.14 167.64)
 		(scale 0.401781)
 		(data "iVBORw0KGgoAAAANSUhEUgAAAOAAAADgCAIAAACVT/22AAAAA3NCSVQICAjb4U/gAAAgAElEQVR4"
@@
 	(symbol
 		(lib_id "Connector:Screw_Terminal_01x01")
-		(at 350.52 176.53 0)
+		(at 349.25 167.64 0)
 		(unit 1)
 		(body_style 1)
@@
 		(dnp yes)
 		(property "Reference" "J6"
-			(at 349.25 173.99 0)
+			(at 347.98 165.1 0)
 			(show_name no)
 			(do_not_autoplace no)
@@
 		)
 		(property "Value" "Screw_Terminal_01x01"
-			(at 353.06 177.7999 0)
+			(at 351.79 168.9099 0)
 			(hide yes)
 			(show_name no)
@@
 		)
 		(property "Footprint" "Bvrny's_library:M8_NutTerminal"
-			(at 350.52 176.53 0)
+			(at 349.25 167.64 0)
 			(hide yes)
 			(show_name no)
@@
 		)
 		(property "Datasheet" ""
-			(at 350.52 176.53 0)
+			(at 349.25 167.64 0)
 			(hide yes)
 			(show_name no)
@@
 		)
 		(property "Description" "Generic screw terminal, single row, 01x01, script generated (kicad-library-utils/schlib/autogen/connector/)"
-			(at 350.52 176.53 0)
+			(at 349.25 167.64 0)
 			(hide yes)
 			(show_name no)
@@
 	)
 	(sheet
-		(at 241.3 114.3)
-		(size 38.1 38.1)
+		(at 240.03 118.11)
+		(size 30.48 22.86)
 		(exclude_from_sim no)
 		(in_bom yes)
@@
 		)
 		(property "Sheetname" "Phase V"
-			(at 241.3 113.5122 0)
+			(at 240.03 117.3222 0)
 			(show_name no)
 			(do_not_autoplace no)
@@
 		)
 		(property "Sheetfile" "PhaseV.kicad_sch"
-			(at 241.3 153.0608 0)
+			(at 240.03 141.6308 0)
 			(hide yes)
 			(show_name no)
@@
 		)
 		(pin "PhaseV_out" output
-			(at 279.4 129.54 0)
+			(at 270.51 129.54 0)
 			(effects
 				(font
@@
 			)
 		)
-		(pin "phV_HS" passive
-			(at 241.3 121.92 180)
-			(effects
-				(font
-					(size 1.27 1.27)
-				)
-				(justify left)
-			)
-		)
-		(pin "phV_HSgate1" passive
-			(at 241.3 129.54 180)
-			(effects
-				(font
-					(size 1.27 1.27)
-				)
-				(justify left)
-			)
-		)
-		(pin "phV_HSgate2" passive
-			(at 241.3 134.62 180)
-			(effects
-				(font
-					(size 1.27 1.27)
-				)
-				(justify left)
-			)
-		)
-		(pin "phV_I+" output
-			(at 241.3 140.97 180)
-			(effects
-				(font
-					(size 1.27 1.27)
-				)
-				(justify left)
-			)
-		)
-		(pin "phV_I-" output
-			(at 241.3 144.78 180)
-			(effects
-				(font
-					(size 1.27 1.27)
-				)
-				(justify left)
-			)
-		)
-		(pin "phV_LSgate1" passive
-			(at 241.3 148.59 180)
-			(effects
-				(font
-					(size 1.27 1.27)
-				)
-				(justify left)
-			)
-		)
-		(pin "phV_LSgate2" passive
-			(at 241.3 132.08 180)
-			(effects
-				(font
-					(size 1.27 1.27)
-				)
-				(justify left)
-			)
-		)
-		(pin "phV_NTCctrl" input
-			(at 241.3 125.73 180)
-			(effects
-				(font
-					(size 1.27 1.27)
-				)
-				(justify left)
-			)
-		)
-		(pin "phV_NTCout" output
-			(at 241.3 118.11 180)
-			(effects
-				(font
-					(size 1.27 1.27)
-				)
-				(justify left)
-			)
-		)
-		(pin "phV_Voltage" output
-			(at 241.3 127 180)
-			(effects
-				(font
-					(size 1.27 1.27)
-				)
-				(justify left)
-			)
-		)
 		(instances
 			(project "PCBA-FLUX-01A"
@@
 	)
 	(sheet
-		(at 241.3 165.1)
-		(size 38.1 38.1)
+		(at 240.03 156.21)
+		(size 30.48 24.13)
 		(exclude_from_sim no)
 		(in_bom yes)
@@
 		)
 		(property "Sheetname" "Phase W"
-			(at 241.3 164.3122 0)
+			(at 240.03 155.4222 0)
 			(show_name no)
 			(do_not_autoplace no)
@@
 		)
 		(property "Sheetfile" "PhaseW.kicad_sch"
-			(at 241.3 203.8608 0)
+			(at 240.03 181.0008 0)
 			(hide yes)
 			(show_name no)
@@
 		)
 		(pin "PhaseW_out" output
-			(at 279.4 176.53 0)
+			(at 270.51 167.64 0)
 			(effects
 				(font
@@
 			)
 		)
-		(pin "phW_HS" passive
-			(at 241.3 168.91 180)
-			(effects
-				(font
-					(size 1.27 1.27)
-				)
-				(justify left)
-			)
-		)
-		(pin "phW_HSgate1" passive
-			(at 241.3 172.72 180)
-			(effects
-				(font
-					(size 1.27 1.27)
-				)
-				(justify left)
-			)
-		)
-		(pin "phW_HSgate2" passive
-			(at 241.3 175.26 180)
-			(effects
-				(font
-					(size 1.27 1.27)
-				)
-				(justify left)
-			)
-		)
-		(pin "phW_I+" output
-			(at 241.3 177.8 180)
-			(effects
-				(font
-					(size 1.27 1.27)
-				)
-				(justify left)
-			)
-		)
-		(pin "phW_I-" output
-			(at 241.3 180.34 180)
-			(effects
-				(font
-					(size 1.27 1.27)
-				)
-				(justify left)
-			)
-		)
-		(pin "phW_LSgate1" passive
-			(at 241.3 184.15 180)
-			(effects
-				(font
-					(size 1.27 1.27)
-				)
-				(justify left)
-			)
-		)
-		(pin "phW_LSgate2" passive
-			(at 241.3 190.5 180)
-			(effects
-				(font
-					(size 1.27 1.27)
-				)
-				(justify left)
-			)
-		)
-		(pin "phW_NTCctrl" input
-			(at 241.3 195.58 180)
-			(effects
-				(font
-					(size 1.27 1.27)
-				)
-				(justify left)
-			)
-		)
-		(pin "phW_NTCout" output
-			(at 241.3 191.77 180)
-			(effects
-				(font
-					(size 1.27 1.27)
-				)
-				(justify left)
-			)
-		)
-		(pin "phW_Voltage" output
-			(at 241.3 187.96 180)
-			(effects
-				(font
-					(size 1.27 1.27)
-				)
-				(justify left)
-			)
-		)
 		(instances
 			(project "PCBA-FLUX-01A"
@@
 		)
 		(pin "phU_NTCctrl" input
-			(at 241.3 87.63 180)
+			(at 241.3 88.9 180)
 			(effects
 				(font
@@
 			(effects
 				(font
-					(size 1.27 1.27)
-				)
-				(justify left)
-			)
-		)
-		(pin "phU_Voltage" output
-			(at 241.3 82.55 180)
-			(effects
-				(font
