File: PCBA-FLUX-01A/_restore_backup_2026-08-26T13-48-18-741/BlockDiagram.kicad_sch (KiCad schematic)
At the start: 47 parts, among them J1 Conn_01x03_Pin, J10 Screw_Terminal_01x01, J11 Conn_01x03_Pin, J12 Conn_01x03_Pin, J13 Conn_01x03_Pin, J14 Conn_01x03_Pin, J15 Conn_01x03_Pin, J16 Conn_01x03_Pin, J17 Conn_01x03_Pin, J18 Conn_01x03_Pin, J19 Conn_01x03_Pin, J2 Conn_01x03_Pin, J20 Conn_01x05_Pin, J21 Conn_01x04_Pin, J22 Conn_01x05_Pin, J23 Conn_01x04_Pin, J24 Conn_01x05_Pin, J25 Conn_01x04_Pin, J26 Screw_Terminal_01x01, J27 Screw_Terminal_01x01, J3 Conn_01x03_Pin, J4 Screw_Terminal_01x01, J5 Screw_Terminal_01x01, J6 Screw_Terminal_01x01, J7 Conn_02x02_Odd_Even, J8 Conn_02x02_Odd_Even, J9 Screw_Terminal_01x01

Commit message: Changing PC
Parts:
- removed C143, C144, C145, C146, C147, C148, C149, C150, C151, C152, C153, C154: 1000uF, Capacitor_THT:CP_Radial_D18.0mm_P7.50mm, symbol Device:C_Polarized
- removed H1, H2, H3, H4, H5, H6, H7, H8: MountingHole, MountingHole_4.3mm_M4_Pad_Via, symbol Mechanical:MountingHole
- removed J1, J11, J12, J13, J14, J15, J16, J17, J18, J19, J2, J3: Conn_01x03_Pin, Connector_PinHeader_2.54mm:PinHeader_1x03_P2.54mm_Vertical, symbol Connector:Conn_01x03_Pin
- removed J10, J26, J27, J4, J5, J6, J9: Screw_Terminal_01x01, Bvrny's_library:M8_NutTerminal, symbol Connector:Screw_Terminal_01x01
- removed J20, J22, J24: Conn_01x05_Pin, Connector_PinHeader_2.54mm:PinHeader_1x05_P2.54mm_Vertical, symbol Connector:Conn_01x05_Pin
- removed J21, J23, J25: Conn_01x04_Pin, Connector_PinHeader_2.54mm:PinHeader_1x04_P2.54mm_Vertical, symbol Connector:Conn_01x04_Pin
- removed J7, J8: Conn_02x02_Odd_Even, Connector_PinHeader_2.54mm:PinHeader_2x02_P2.54mm_Vertical, symbol Connector_Generic:Conn_02x02_Odd_Even
Other:
- removed sheet Phase U
- removed sheet Phase V
- removed sheet Phase W
- note removed: "Board connectors for power to Vector"
- note removed: "Board connectors to Vector"
- note removed: "High current connectors"
- note removed: "Inverter"
- note removed: "Power input connectors"
