File: PCBA-FLUX-01A/_restore_backup_2026-08-26T13-48-18-741/PhaseU.kicad_sch (KiCad schematic)
At the start: 47 parts, among them J1 Conn_01x03_Pin, J10 Screw_Terminal_01x01, J11 Conn_01x03_Pin, J12 Conn_01x03_Pin, J13 Conn_01x03_Pin, J14 Conn_01x03_Pin, J15 Conn_01x03_Pin, J16 Conn_01x03_Pin, J17 Conn_01x03_Pin, J18 Conn_01x03_Pin, J19 Conn_01x03_Pin, J2 Conn_01x03_Pin, J20 Conn_01x05_Pin, J21 Conn_01x04_Pin, J22 Conn_01x05_Pin, J23 Conn_01x04_Pin, J24 Conn_01x05_Pin, J25 Conn_01x04_Pin, J26 Screw_Terminal_01x01, J27 Screw_Terminal_01x01, J3 Conn_01x03_Pin, J4 Screw_Terminal_01x01, J5 Screw_Terminal_01x01, J6 Screw_Terminal_01x01, J7 Conn_02x02_Odd_Even, J8 Conn_02x02_Odd_Even, J9 Screw_Terminal_01x01

Commit message: Changing PC
Parts:
- removed C143, C144, C145, C146, C147, C148, C149, C150, C151, C152, C153, C154: 1000uF, Capacitor_THT:CP_Radial_D18.0mm_P7.50mm, symbol Device:C_Polarized
- removed H1, H2, H3, H4, H5, H6, H7, H8: MountingHole, MountingHole_4.3mm_M4_Pad_Via, symbol Mechanical:MountingHole
- removed J1, J11, J12, J13, J14, J15, J16, J17, J18, J19, J2, J3: Conn_01x03_Pin, Connector_PinHeader_2.54mm:PinHeader_1x03_P2.54mm_Vertical, symbol Connector:Conn_01x03_Pin
- removed J10, J26, J27, J4, J5, J6, J9: Screw_Terminal_01x01, Bvrny's_library:M8_NutTerminal, symbol Connector:Screw_Terminal_01x01
- removed J20, J22, J24: Conn_01x05_Pin, Connector_PinHeader_2.54mm:PinHeader_1x05_P2.54mm_Vertical, symbol Connector:Conn_01x05_Pin
- removed J21, J23, J25: Conn_01x04_Pin, Connector_PinHeader_2.54mm:PinHeader_1x04_P2.54mm_Vertical, symbol Connector:Conn_01x04_Pin
- removed J7, J8: Conn_02x02_Odd_Even, Connector_PinHeader_2.54mm:PinHeader_2x02_P2.54mm_Vertical, symbol Connector_Generic:Conn_02x02_Odd_Even
- added C104: C, Capacitor_THT:C_Rect_L9.0mm_W6.4mm_P7.50mm_MKT, symbol Device:C
- added C48: 100nF, Capacitor_SMD:C_0402_1005Metric, symbol Device:C
- added C56: 3.3nF, Capacitor_SMD:C_0603_1608Metric, symbol Device:C
- added C99: 10nF, Capacitor_SMD:C_0603_1608Metric, symbol Device:C
- added D2, D3, D4, D5: SS34, Diode_SMD:D_SMA, symbol Device:D_Schottky
- added Q18: BC860C, Package_TO_SOT_SMD:SOT-23, symbol Simulation_SPICE:PNP
- added Q2, Q3, Q4, Q5: IPT015N10N5, Package_TO_SOT_SMD:Infineon_PG-HSOF-8-1_ThermalVias, symbol Bvrny's_library:IPT015N10N5
- added R13, R14, R4, R5: 1R, Resistor_SMD:R_1206_3216Metric, symbol Device:R
- added R15, R16, R6, R7: 3R3, Resistor_SMD:R_1206_3216Metric, symbol Device:R
- added R18, R19, R8, R9: 10k, Resistor_SMD:R_1206_3216Metric, symbol Device:R
- added R20: 0.1mR, Bvrny's_library:R5930, symbol Device:R_Shunt
- added R21: 2K2, Resistor_SMD:R_0603_1608Metric, symbol Device:R
- added R22: 560R, Resistor_SMD:R_0603_1608Metric, symbol Device:R
- added R23: 0R, Resistor_SMD:R_0603_1608Metric, symbol Device:R
- added R25: 10K, Resistor_SMD:R_0603_1608Metric, symbol Device:R
- added R26, R27: 51k, Resistor_SMD:R_0805_2012Metric, symbol Device:R
- added R34: 4k7, Resistor_SMD:R_0805_2012Metric, symbol Device:R
- added R76, R77, R78, R79: 10R, Resistor_SMD:R_0805_2012Metric, symbol Device:R
- added R90: R, Resistor_SMD:R_1218_3246Metric, symbol Device:R
- added R93: 18k, Resistor_SMD:R_0603_1608Metric, symbol Synapse:R
- added TH1: NCP18XH103F03RB, Resistor_SMD:R_0603_1608Metric, symbol Device:Thermistor_NTC
Connections:
- net +3.3VA: now also Q18.3 (E), R23.1, R93.1
- net +VSYS: now also Q2.3, Q4.3
- net GND: now also C104.2, C48.2, C56.2, Q3.2, Q5.2, R19.2, R34.2, R9.2, TH1.2
- new net: D4.2 (A), Q4.1, R15.2, R18.1
- new net: Q18.2 (B), R21.2
- new net: R22.2, R25.1, R93.2, TH1.1
- new net: D4.1 (K), R13.2
- new net: D5.2 (A), Q5.1, R16.2, R19.1
- new net: D2.2 (A), Q2.1, R6.2, R8.1
- new net: Q18.1 (C), R22.1, R23.2
- new net: D3.2 (A), Q3.1, R7.2, R9.1
- new net: D3.1 (K), R5.2
- new net: C104.1, R90.2
- new net: R26.2, R27.1
- new net: D2.1 (K), R4.2
- new net: D5.1 (K), R14.2
- new net PhaseU_out: R20.4, R26.1
- new net phU_HS: Q2.2, Q3.3, Q4.2, Q5.3, R18.2, R20.1, R8.2, R90.1
- new net phU_HSgate1: R4.1, R6.1
- new net phU_HSgate2: R13.1, R15.1
- new net phU_I+: C99.2, R78.2, R79.2
- new net phU_I-: C99.1, R76.2, R77.2
- new net phU_LSgate1: R5.1, R7.1
- new net phU_LSgate2: R14.1, R16.1
- new net phU_NTCctrl: R21.1
- new net phU_NTCout: C48.1, R25.2
- new net phU_Shunt+: R20.2, R78.1, R79.1
- new net phU_Shunt-: R20.3, R76.1, R77.1
- new net phU_Voltage: C56.1, R27.2, R34.1
Other:
- removed sheet Phase U
- removed sheet Phase V
- removed sheet Phase W
- note added: "Bridge"
- note added: "Phase Temp"
- note removed: "Board connectors for power to Vector"
- note removed: "Board connectors to Vector"
- note removed: "High current connectors"
- note removed: "Inverter"
- note removed: "Power input connectors"
