File: PCBA-FLUX-01A/_restore_backup_2026-08-26T13-48-18-741/PhaseV.kicad_sch (KiCad schematic)
At the start: 47 parts, among them J1 Conn_01x03_Pin, J10 Screw_Terminal_01x01, J11 Conn_01x03_Pin, J12 Conn_01x03_Pin, J13 Conn_01x03_Pin, J14 Conn_01x03_Pin, J15 Conn_01x03_Pin, J16 Conn_01x03_Pin, J17 Conn_01x03_Pin, J18 Conn_01x03_Pin, J19 Conn_01x03_Pin, J2 Conn_01x03_Pin, J20 Conn_01x05_Pin, J21 Conn_01x04_Pin, J22 Conn_01x05_Pin, J23 Conn_01x04_Pin, J24 Conn_01x05_Pin, J25 Conn_01x04_Pin, J26 Screw_Terminal_01x01, J27 Screw_Terminal_01x01, J3 Conn_01x03_Pin, J4 Screw_Terminal_01x01, J5 Screw_Terminal_01x01, J6 Screw_Terminal_01x01, J7 Conn_02x02_Odd_Even, J8 Conn_02x02_Odd_Even, J9 Screw_Terminal_01x01

Commit message: Changing PC
Parts:
- removed C143, C144, C145, C146, C147, C148, C149, C150, C151, C152, C153, C154: 1000uF, Capacitor_THT:CP_Radial_D18.0mm_P7.50mm, symbol Device:C_Polarized
- removed H1, H2, H3, H4, H5, H6, H7, H8: MountingHole, MountingHole_4.3mm_M4_Pad_Via, symbol Mechanical:MountingHole
- removed J1, J11, J12, J13, J14, J15, J16, J17, J18, J19, J2, J3: Conn_01x03_Pin, Connector_PinHeader_2.54mm:PinHeader_1x03_P2.54mm_Vertical, symbol Connector:Conn_01x03_Pin
- removed J10, J26, J27, J4, J5, J6, J9: Screw_Terminal_01x01, Bvrny's_library:M8_NutTerminal, symbol Connector:Screw_Terminal_01x01
- removed J20, J22, J24: Conn_01x05_Pin, Connector_PinHeader_2.54mm:PinHeader_1x05_P2.54mm_Vertical, symbol Connector:Conn_01x05_Pin
- removed J21, J23, J25: Conn_01x04_Pin, Connector_PinHeader_2.54mm:PinHeader_1x04_P2.54mm_Vertical, symbol Connector:Conn_01x04_Pin
- removed J7, J8: Conn_02x02_Odd_Even, Connector_PinHeader_2.54mm:PinHeader_2x02_P2.54mm_Vertical, symbol Connector_Generic:Conn_02x02_Odd_Even
- added C100: 10nF, Capacitor_SMD:C_0603_1608Metric, symbol Device:C
- added C105: C, Capacitor_THT:C_Rect_L9.0mm_W6.4mm_P7.50mm_MKT, symbol Device:C
- added C57: 3.3nF, Capacitor_SMD:C_0603_1608Metric, symbol Device:C
- added C63: 100nF, Capacitor_SMD:C_0402_1005Metric, symbol Device:C
- added D6, D7, D8, D9: SS34, Diode_SMD:D_SMA, symbol Device:D_Schottky
- added Q19: BC860C, Package_TO_SOT_SMD:SOT-23, symbol Simulation_SPICE:PNP
- added Q6, Q7, Q8, Q9: IPT015N10N5, Package_TO_SOT_SMD:Infineon_PG-HSOF-8-1_ThermalVias, symbol Bvrny's_library:IPT015N10N5
- added R28, R29, R37, R38: 1R, Resistor_SMD:R_1206_3216Metric, symbol Device:R
- added R30, R31, R39, R40: 3R3, Resistor_SMD:R_1206_3216Metric, symbol Device:R
- added R32, R33, R41, R42: 10k, Resistor_SMD:R_1206_3216Metric, symbol Device:R
- added R35, R36: 51k, Resistor_SMD:R_0805_2012Metric, symbol Device:R
- added R43: 4k7, Resistor_SMD:R_0805_2012Metric, symbol Device:R
- added R44: 0.1mR, Bvrny's_library:R5930, symbol Device:R_Shunt
- added R45: 2K2, Resistor_SMD:R_0603_1608Metric, symbol Device:R
- added R46: 560R, Resistor_SMD:R_0603_1608Metric, symbol Device:R
- added R47: 0R, Resistor_SMD:R_0603_1608Metric, symbol Device:R
- added R48: 10K, Resistor_SMD:R_0603_1608Metric, symbol Device:R
- added R80, R81, R82, R83: 10R, Resistor_SMD:R_0805_2012Metric, symbol Device:R
- added R91: R, Resistor_SMD:R_1218_3246Metric, symbol Device:R
- added R94: 18k, Resistor_SMD:R_0603_1608Metric, symbol Synapse:R
- added TH2: NCP18XH103F03RB, Resistor_SMD:R_0603_1608Metric, symbol Device:Thermistor_NTC
Connections:
- net +3.3VA: now also Q19.3 (E), R47.1, R94.1
- net +VSYS: now also Q6.3, Q8.3
- net GND: now also C105.2, C57.2, C63.2, Q7.2, Q9.2, R33.2, R42.2, R43.2, TH2.2
- new net: C105.1, R91.2
- new net: Q19.1 (C), R46.1, R47.2
- new net: D9.2 (A), Q9.1, R40.2, R42.1
- new net: D6.2 (A), Q6.1, R30.2, R32.1
- new net: D8.2 (A), Q8.1, R39.2, R41.1
- new net: D6.1 (K), R28.2
- new net: Q19.2 (B), R45.2
- new net: D7.2 (A), Q7.1, R31.2, R33.1
- new net: D9.1 (K), R38.2
- new net: R46.2, R48.1, R94.2, TH2.1
- new net: D8.1 (K), R37.2
- new net: R35.2, R36.1
- new net: D7.1 (K), R29.2
- new net PhaseV_out: R35.1, R44.4
- new net phV_HS: Q6.2, Q7.3, Q8.2, Q9.3, R32.2, R41.2, R44.1, R91.1
- new net phV_HSgate1: R28.1, R30.1
- new net phV_HSgate2: R37.1, R39.1
- new net phV_I+: C100.2, R80.2, R81.2
- new net phV_I-: C100.1, R82.2, R83.2
- new net phV_LSgate1: R29.1, R31.1
- new net phV_LSgate2: R38.1, R40.1
- new net phV_NTCctrl: R45.1
- new net phV_NTCout: C63.1, R48.2
- new net phV_Shunt+: R44.2, R80.1, R81.1
- new net phV_Shunt-: R44.3, R82.1, R83.1
- new net phV_Voltage: C57.1, R36.2, R43.1
Other:
- removed sheet Phase U
- removed sheet Phase V
- removed sheet Phase W
- note added: "Gate driver & bridge"
- note added: "Phase Temp"
- note removed: "Board connectors for power to Vector"
- note removed: "Board connectors to Vector"
- note removed: "High current connectors"
- note removed: "Inverter"
- note removed: "Power input connectors"
