File: PCBA-FLUX-01A/_restore_backup_2026-08-26T13-48-18-741/PhaseW.kicad_sch (KiCad schematic)
At the start: 47 parts, among them J1 Conn_01x03_Pin, J10 Screw_Terminal_01x01, J11 Conn_01x03_Pin, J12 Conn_01x03_Pin, J13 Conn_01x03_Pin, J14 Conn_01x03_Pin, J15 Conn_01x03_Pin, J16 Conn_01x03_Pin, J17 Conn_01x03_Pin, J18 Conn_01x03_Pin, J19 Conn_01x03_Pin, J2 Conn_01x03_Pin, J20 Conn_01x05_Pin, J21 Conn_01x04_Pin, J22 Conn_01x05_Pin, J23 Conn_01x04_Pin, J24 Conn_01x05_Pin, J25 Conn_01x04_Pin, J26 Screw_Terminal_01x01, J27 Screw_Terminal_01x01, J3 Conn_01x03_Pin, J4 Screw_Terminal_01x01, J5 Screw_Terminal_01x01, J6 Screw_Terminal_01x01, J7 Conn_02x02_Odd_Even, J8 Conn_02x02_Odd_Even, J9 Screw_Terminal_01x01

Commit message: Changing PC
Parts:
- removed C143, C144, C145, C146, C147, C148, C149, C150, C151, C152, C153, C154: 1000uF, Capacitor_THT:CP_Radial_D18.0mm_P7.50mm, symbol Device:C_Polarized
- removed H1, H2, H3, H4, H5, H6, H7, H8: MountingHole, MountingHole_4.3mm_M4_Pad_Via, symbol Mechanical:MountingHole
- removed J1, J11, J12, J13, J14, J15, J16, J17, J18, J19, J2, J3: Conn_01x03_Pin, Connector_PinHeader_2.54mm:PinHeader_1x03_P2.54mm_Vertical, symbol Connector:Conn_01x03_Pin
- removed J10, J26, J27, J4, J5, J6, J9: Screw_Terminal_01x01, Bvrny's_library:M8_NutTerminal, symbol Connector:Screw_Terminal_01x01
- removed J20, J22, J24: Conn_01x05_Pin, Connector_PinHeader_2.54mm:PinHeader_1x05_P2.54mm_Vertical, symbol Connector:Conn_01x05_Pin
- removed J21, J23, J25: Conn_01x04_Pin, Connector_PinHeader_2.54mm:PinHeader_1x04_P2.54mm_Vertical, symbol Connector:Conn_01x04_Pin
- removed J7, J8: Conn_02x02_Odd_Even, Connector_PinHeader_2.54mm:PinHeader_2x02_P2.54mm_Vertical, symbol Connector_Generic:Conn_02x02_Odd_Even
- added C101: 10nF, Capacitor_SMD:C_0603_1608Metric, symbol Device:C
- added C106: C, Capacitor_THT:C_Rect_L9.0mm_W6.4mm_P7.50mm_MKT, symbol Device:C
- added C130, C132, C134, C136, C138: 10uF, Capacitor_SMD:C_1210_3225Metric, symbol Device:C
- added C139, C78, C79, C80, C82: 100nF, Capacitor_SMD:C_0805_2012Metric, symbol Device:C
- added C58: 3.3nF, Capacitor_SMD:C_0603_1608Metric, symbol Device:C
- added C81: 100nF, Capacitor_SMD:C_0402_1005Metric, symbol Device:C
- added D10, D11, D12, D13: SS34, Diode_SMD:D_SMA, symbol Device:D_Schottky
- added Q10, Q11, Q12, Q13: IPT015N10N5, Package_TO_SOT_SMD:Infineon_PG-HSOF-8-1_ThermalVias, symbol Bvrny's_library:IPT015N10N5
- added Q20: BC860C, Package_TO_SOT_SMD:SOT-23, symbol Simulation_SPICE:PNP
- added R49, R50: 51k, Resistor_SMD:R_0805_2012Metric, symbol Device:R
- added R51: 4k7, Resistor_SMD:R_0805_2012Metric, symbol Device:R
- added R52, R53, R61, R62: 1R, Resistor_SMD:R_1206_3216Metric, symbol Device:R
- added R54, R55, R63, R64: 3R3, Resistor_SMD:R_1206_3216Metric, symbol Device:R
- added R56, R57, R65, R66: 10k, Resistor_SMD:R_1206_3216Metric, symbol Device:R
- added R68: 0.1mR, Bvrny's_library:R5930, symbol Device:R_Shunt
- added R69: 2K2, Resistor_SMD:R_0603_1608Metric, symbol Device:R
- added R70: 560R, Resistor_SMD:R_0603_1608Metric, symbol Device:R
- added R71: 0R, Resistor_SMD:R_0603_1608Metric, symbol Device:R
- added R72: 10K, Resistor_SMD:R_0603_1608Metric, symbol Device:R
- added R84, R85, R86, R87: 10R, Resistor_SMD:R_0805_2012Metric, symbol Device:R
- added R92: R, Resistor_SMD:R_1218_3246Metric, symbol Device:R
- added R95: 18k, Resistor_SMD:R_0603_1608Metric, symbol Synapse:R
- added TH3: NCP18XH103F03RB, Resistor_SMD:R_0603_1608Metric, symbol Device:Thermistor_NTC
Connections:
- net +3.3VA: now also Q20.3 (E), R71.1, R95.1
- net +VSYS: now also C130.1, C132.1, C134.1, C136.1, C138.1, C139.1, C78.1, C79.1, C80.1, C82.1, Q10.3, Q12.3
- net GND: now also C106.2, C130.2, C132.2, C134.2, C136.2, C138.2, C139.2, C58.2, C78.2, C79.2, C80.2, C81.2, C82.2, Q11.2, Q13.2, R51.2, R57.2, R66.2, TH3.2
- new net: D12.2 (A), Q12.1, R63.2, R65.1
- new net: R70.2, R72.1, R95.2, TH3.1
- new net: D13.2 (A), Q13.1, R64.2, R66.1
- new net: D11.1 (K), R53.2
- new net: D10.1 (K), R52.2
- new net: D10.2 (A), Q10.1, R54.2, R56.1
- new net: C106.1, R92.2
- new net: Q20.1 (C), R70.1, R71.2
- new net: Q20.2 (B), R69.2
- new net: D12.1 (K), R61.2
- new net: D11.2 (A), Q11.1, R55.2, R57.1
- new net: D13.1 (K), R62.2
- new net: R49.2, R50.1
- new net PhaseW_out: R49.1, R68.4
- new net phW_HS: Q10.2, Q11.3, Q12.2, Q13.3, R56.2, R65.2, R68.1, R92.1
- new net phW_HSgate1: R52.1, R54.1
- new net phW_HSgate2: R61.1, R63.1
- new net phW_I+: C101.2, R84.2, R85.2
- new net phW_I-: C101.1, R86.2, R87.2
- new net phW_LSgate1: R53.1, R55.1
- new net phW_LSgate2: R62.1, R64.1
- new net phW_NTCctrl: R69.1
- new net phW_NTCout: C81.1, R72.2
- new net phW_Shunt+: R68.2, R84.1, R85.1
- new net phW_Shunt-: R68.3, R86.1, R87.1
- new net phW_Voltage: C58.1, R50.2, R51.1
Other:
- removed sheet Phase U
- removed sheet Phase V
- removed sheet Phase W
- note added: "DC-Link"
- note added: "Gate driver & bridge"
- note added: "Phase Temp"
- note removed: "Board connectors for power to Vector"
- note removed: "Board connectors to Vector"
- note removed: "High current connectors"
- note removed: "Inverter"
- note removed: "Power input connectors"
