File: PCBA-FLUX-01A/_restore_backup_2026-08-26T13-48-18-741/ProjectArchitecture.kicad_sch (KiCad schematic)
At the start: 47 parts, among them J1 Conn_01x03_Pin, J10 Screw_Terminal_01x01, J11 Conn_01x03_Pin, J12 Conn_01x03_Pin, J13 Conn_01x03_Pin, J14 Conn_01x03_Pin, J15 Conn_01x03_Pin, J16 Conn_01x03_Pin, J17 Conn_01x03_Pin, J18 Conn_01x03_Pin, J19 Conn_01x03_Pin, J2 Conn_01x03_Pin, J20 Conn_01x05_Pin, J21 Conn_01x04_Pin, J22 Conn_01x05_Pin, J23 Conn_01x04_Pin, J24 Conn_01x05_Pin, J25 Conn_01x04_Pin, J26 Screw_Terminal_01x01, J27 Screw_Terminal_01x01, J3 Conn_01x03_Pin, J4 Screw_Terminal_01x01, J5 Screw_Terminal_01x01, J6 Screw_Terminal_01x01, J7 Conn_02x02_Odd_Even, J8 Conn_02x02_Odd_Even, J9 Screw_Terminal_01x01

Commit message: Changing PC
Parts:
- removed H1, H2, H3, H4, H5, H6, H7, H8: MountingHole, MountingHole_4.3mm_M4_Pad_Via, symbol Mechanical:MountingHole
